Commit message: demo node compiles ...

File: yumi_description/urdf/yumi_servo_gripper.gazebo.xacro (robot description, xacro)
@@ -2,4 +2,12 @@
 <robot name="yumi_servo_gripper" xmlns:xacro="http://www.ros.org/wiki/xacro">
   <xacro:macro name="yumi_servo_gripper_gazebo" params="name">
+  <!-- Plugin for the mimic o/c joint - AFAIK, that shouldn't be necessary any more starting with Gazebo 3.0 -->
+    <gazebo>
+      <plugin name="mimic_plugin" filename="libgazebo_mimic_plugin.so">
+       <joint>${name}_joint</joint>
+        <mimicJoint>${name}_joint_m</mimicJoint>
+        <multiplier>1.0</multiplier>
+      </plugin>
+    </gazebo>
     <!-- body -->
     <gazebo reference="${name}_base">

File: yumi_description/urdf/yumi_servo_gripper.transmission.xacro (robot description, xacro)
@@ -2,10 +2,10 @@
 <robot name="yumi_servo_gripper" xmlns:xacro="http://www.ros.org/wiki/xacro">
   <xacro:macro name="yumi_servo_gripper_transmission" params="name hardware_interface">
-   <transmission name="${name}_tran_1">
+   <transmission name="${name}_tran">
       <type>transmission_interface/SimpleTransmission</type>
-      <joint name="${name}_joint_1">
+      <joint name="${name}_joint">
 	<hardwareInterface>${hardware_interface}</hardwareInterface>
       </joint>
-      <actuator name="${name}_motor_1">
+      <actuator name="${name}_motor">
 	<hardwareInterface>${hardware_interface}</hardwareInterface>
 	<mechanicalReduction>1</mechanicalReduction>
