Commit message: some progress on the urdfs

File: yumi_description/urdf/materials.xacro (robot description, xacro)
@@ -11,5 +11,11 @@
   </material>
   <material name="Grey">
-    <color rgba="0.2 0.2 0.2 1.0"/>
+    <color rgba="0.5 0.5 0.5 1.0"/>
+  </material>
+  <material name="Light_Grey">
+    <color rgba="0.8 0.8 0.8 1.0"/>
+  </material>
+  <material name="Ivory">
+    <color rgba="1.0 1.0 0.94 1.0"/>
   </material>
   <material name="Orange">

File: yumi_description/urdf/yumi.gazebo.xacro (robot description, xacro)
@@ -1,50 +1,8 @@
 <?xml version="1.0"?>
-<robot name="lbr_iiwa" xmlns:xacro="http://www.ros.org/wiki/xacro">
-  <xacro:macro name="lbr_iiwa_gazebo" params="name">
-    <!-- Link0 -->
-    <gazebo reference="${name}_link_0">
-      <material>Gazebo/Grey</material>
-      <mu1>0.2</mu1>
-      <mu2>0.2</mu2>
-    </gazebo>
-    <!-- Link1 -->
-    <gazebo reference="${name}_link_1">
-      <material>Gazebo/Orange</material>
-      <mu1>0.2</mu1>
-      <mu2>0.2</mu2>
-    </gazebo>
-    <!-- Link2 -->
-    <gazebo reference="${name}_link_2">
-      <material>Gazebo/Orange</material>
-      <mu1>0.2</mu1>
-      <mu2>0.2</mu2>
-    </gazebo>
-    <!-- Link3 -->
-    <gazebo reference="${name}_link_3">
-      <material>Gazebo/Orange</material>
-      <mu1>0.2</mu1>
-      <mu2>0.2</mu2>
-    </gazebo>
-    <!-- Link4 -->
-    <gazebo reference="${name}_link_4">
-      <material>Gazebo/Orange</material>
-      <mu1>0.2</mu1>
-      <mu2>0.2</mu2>
-    </gazebo>
-    <!-- Link5 -->
-    <gazebo reference="${name}_link_5">
-      <material>Gazebo/Orange</material>
-      <mu1>0.2</mu1>
-      <mu2>0.2</mu2>
-    </gazebo>
-    <!-- Link6 -->
-    <gazebo reference="${name}_link_6">
-      <material>Gazebo/Orange</material>
-      <mu1>0.2</mu1>
-      <mu2>0.2</mu2>
-    </gazebo>
-    <!-- Link7 -->
-    <gazebo reference="${name}_link_7">
-      <material>Gazebo/Grey</material>
+<robot name="yumi" xmlns:xacro="http://www.ros.org/wiki/xacro">
+  <xacro:macro name="yumi_gazebo" params="name">
+    <!-- body -->
+    <gazebo reference="${name}_body">
+      <material>Gazebo/Ivory</material>
       <mu1>0.2</mu1>
       <mu2>0.2</mu2>

File: yumi_description/urdf/yumi.transmission.xacro (robot description, xacro)
@@ -1,71 +1,141 @@
 <?xml version="1.0"?>
-<robot name="lbr_iiwa" xmlns:xacro="http://www.ros.org/wiki/xacro">
-  <xacro:macro name="lbr_iiwa_transmission" params="name hardware_interface">
-    <transmission name="${name}_tran_1">
+<robot name="yumi" xmlns:xacro="http://www.ros.org/wiki/xacro">
+  <xacro:macro name="yumi_transmission" params="name hardware_interface">
+    <transmission name="${name}_tran_1_r">
       <type>transmission_interface/SimpleTransmission</type>
-      <joint name="${name}_joint_1">
+      <joint name="${name}_joint_1_r">
 	<hardwareInterface>${hardware_interface}</hardwareInterface>
       </joint>
-      <actuator name="${name}_motor_1">
+      <actuator name="${name}_motor_1_r">
 	<hardwareInterface>${hardware_interface}</hardwareInterface>
 	<mechanicalReduction>1</mechanicalReduction>
       </actuator>
     </transmission>
-    <transmission name="${name}_tran_2">
+    <transmission name="${name}_tran_2_r">
       <type>transmission_interface/SimpleTransmission</type>
-      <joint name="${name}_joint_2">
+      <joint name="${name}_joint_2_r">
 	<hardwareInterface>${hardware_interface}</hardwareInterface>
       </joint>
-      <actuator name="${name}_motor_2">
+      <actuator name="${name}_motor_2_r">
 	<hardwareInterface>${hardware_interface}</hardwareInterface>
 	<mechanicalReduction>1</mechanicalReduction>
       </actuator>
     </transmission>
-    <transmission name="${name}_tran_3">
+    <transmission name="${name}_tran_3_r">
       <type>transmission_interface/SimpleTransmission</type>
-      <joint name="${name}_joint_3">
+      <joint name="${name}_joint_3_r">
 	<hardwareInterface>${hardware_interface}</hardwareInterface>
       </joint>
-      <actuator name="${name}_motor_3">
+      <actuator name="${name}_motor_3_r">
 	<hardwareInterface>${hardware_interface}</hardwareInterface>
 	<mechanicalReduction>1</mechanicalReduction>
       </actuator>
     </transmission>
-    <transmission name="${name}_tran_4">
+    <transmission name="${name}_tran_4_r">
       <type>transmission_interface/SimpleTransmission</type>
-      <joint name="${name}_joint_4">
+      <joint name="${name}_joint_4_r">
 	<hardwareInterface>${hardware_interface}</hardwareInterface>
       </joint>
-      <actuator name="${name}_motor_4">
+      <actuator name="${name}_motor_4_r">
 	<hardwareInterface>${hardware_interface}</hardwareInterface>
 	<mechanicalReduction>1</mechanicalReduction>
       </actuator>
     </transmission>
-    <transmission name="${name}_tran_5">
+    <transmission name="${name}_tran_5_r">
       <type>transmission_interface/SimpleTransmission</type>
-      <joint name="${name}_joint_5">
+      <joint name="${name}_joint_5_r">
 	<hardwareInterface>${hardware_interface}</hardwareInterface>
       </joint>
-      <actuator name="${name}_motor_5">
+      <actuator name="${name}_motor_5_r">
 	<hardwareInterface>${hardware_interface}</hardwareInterface>
 	<mechanicalReduction>1</mechanicalReduction>
       </actuator>
     </transmission>
-    <transmission name="${name}_tran_6">
+    <transmission name="${name}_tran_6_r">
       <type>transmission_interface/SimpleTransmission</type>
-      <joint name="${name}_joint_6">
+      <joint name="${name}_joint_6_r">
 	<hardwareInterface>${hardware_interface}</hardwareInterface>
       </joint>
-      <actuator name="${name}_motor_6">
+      <actuator name="${name}_motor_6_r">
 	<hardwareInterface>${hardware_interface}</hardwareInterface>
 	<mechanicalReduction>1</mechanicalReduction>
       </actuator>
     </transmission>
-    <transmission name="${name}_tran_7">
+    <transmission name="${name}_tran_7_r">
       <type>transmission_interface/SimpleTransmission</type>
-      <joint name="${name}_joint_7">
+      <joint name="${name}_joint_7_r">
 	<hardwareInterface>${hardware_interface}</hardwareInterface>
       </joint>
-      <actuator name="${name}_motor_7">
+      <actuator name="${name}_motor_7_r">
+	<hardwareInterface>${hardware_interface}</hardwareInterface>
+	<mechanicalReduction>1</mechanicalReduction>
+      </actuator>
+    </transmission>
+    <transmission name="${name}_tran_1_l">
+      <type>transmission_interface/SimpleTransmission</type>
+      <joint name="${name}_joint_1_l">
+	<hardwareInterface>${hardware_interface}</hardwareInterface>
+      </joint>
+      <actuator name="${name}_motor_1_l">
+	<hardwareInterface>${hardware_interface}</hardwareInterface>
+	<mechanicalReduction>1</mechanicalReduction>
+      </actuator>
+    </transmission>
+    <transmission name="${name}_tran_2_l">
+      <type>transmission_interface/SimpleTransmission</type>
+      <joint name="${name}_joint_2_l">
+	<hardwareInterface>${hardware_interface}</hardwareInterface>
+      </joint>
+      <actuator name="${name}_motor_2_l">
+	<hardwareInterface>${hardware_interface}</hardwareInterface>
+	<mechanicalReduction>1</mechanicalReduction>
+      </actuator>
+    </transmission>
+    <transmission name="${name}_tran_3_l">
+      <type>transmission_interface/SimpleTransmission</type>
+      <joint name="${name}_joint_3_l">
+	<hardwareInterface>${hardware_interface}</hardwareInterface>
+      </joint>
+      <actuator name="${name}_motor_3_l">
+	<hardwareInterface>${hardware_interface}</hardwareInterface>
+	<mechanicalReduction>1</mechanicalReduction>
+      </actuator>
+    </transmission>
+    <transmission name="${name}_tran_4_l">
+      <type>transmission_interface/SimpleTransmission</type>
+      <joint name="${name}_joint_4_l">
+	<hardwareInterface>${hardware_interface}</hardwareInterface>
+      </joint>
+      <actuator name="${name}_motor_4_l">
+	<hardwareInterface>${hardware_interface}</hardwareInterface>
+	<mechanicalReduction>1</mechanicalReduction>
+      </actuator>
+    </transmission>
+    <transmission name="${name}_tran_5_l">
+      <type>transmission_interface/SimpleTransmission</type>
+      <joint name="${name}_joint_5_l">
+	<hardwareInterface>${hardware_interface}</hardwareInterface>
+      </joint>
+      <actuator name="${name}_motor_5_l">
+	<hardwareInterface>${hardware_interface}</hardwareInterface>
+	<mechanicalReduction>1</mechanicalReduction>
+      </actuator>
+    </transmission>
+    <transmission name="${name}_tran_6_l">
+      <type>transmission_interface/SimpleTransmission</type>
+      <joint name="${name}_joint_6_l">
+	<hardwareInterface>${hardware_interface}</hardwareInterface>
+      </joint>
+      <actuator name="${name}_motor_6_l">
+	<hardwareInterface>${hardware_interface}</hardwareInterface>
+	<mechanicalReduction>1</mechanicalReduction>
+      </actuator>
+    </transmission>
+    <transmission name="${name}_tran_7_l">
+      <type>transmission_interface/SimpleTransmission</type>
+      <joint name="${name}_joint_7_l">
+	<hardwareInterface>${hardware_interface}</hardwareInterface>
+      </joint>
+      <actuator name="${name}_motor_7_l">
 	<hardwareInterface>${hardware_interface}</hardwareInterface>
 	<mechanicalReduction>1</mechanicalReduction>

File: yumi_description/urdf/yumi.urdf.xacro (robot description, xacro)
@@ -1,15 +1,15 @@
 <?xml version="1.0"?>
-<robot name="lbr_iiwa" xmlns:xacro="http://www.ros.org/wiki/xacro">
+<robot name="yumi" xmlns:xacro="http://www.ros.org/wiki/xacro">
   <!-- Import Rviz colors -->
-  <xacro:include filename="$(find lbr_iiwa_description)/urdf/materials.xacro" />
+  <xacro:include filename="$(find yumi_description)/urdf/materials.xacro" />
   <!--Import the lbr iiwa macro -->
-  <xacro:include filename="$(find lbr_iiwa_description)/urdf/lbr_iiwa.xacro"/>
+  <xacro:include filename="$(find yumi_description)/urdf/yumi.xacro"/>
  <!-- Import Gazebo plugins -->
-  <xacro:include filename="$(find lbr_iiwa_description)/gazebo/gazebo.urdf.xacro"/>
+  <xacro:include filename="$(find yumi_description)/gazebo/gazebo.urdf.xacro"/>
   <!-- Fix to world just for testing -->
   <link name="world"/>
-  <!--lbr-->
-  <xacro:lbr_iiwa name="lbr_iiwa" hardware_interface="$(arg prefix)" parent="world">
-    <origin xyz="0 0 0.0" rpy="0 0 0" />
-  </xacro:lbr_iiwa>
+  <!--yumi-->
+  <xacro:yumi name="yumi" hardware_interface="$(arg prefix)" parent="world">
+    <origin xyz="0 0 0.1" rpy="0 0 0" />
+  </xacro:yumi>
 </robot>
