Commit message: some progress on the urdfs

File: yumi_description/urdf/yumi.xacro (robot description, xacro)
@@ -1,10 +1,10 @@
 <?xml version="1.0"?>
-<robot name="lbr_iiwa" xmlns:xacro="http://www.ros.org/wiki/xacro">
+<robot name="yumi" xmlns:xacro="http://www.ros.org/wiki/xacro">
   <!-- Import all Gazebo-customization elements, including Gazebo colors -->
-  <xacro:include filename="$(find lbr_iiwa_description)/urdf/lbr_iiwa.gazebo.xacro" />
+  <xacro:include filename="$(find yumi_description)/urdf/yumi.gazebo.xacro" />
   <!-- Import Transmissions -->
-  <xacro:include filename="$(find lbr_iiwa_description)/urdf/lbr_iiwa.transmission.xacro" />
+  <xacro:include filename="$(find yumi_description)/urdf/yumi.transmission.xacro" />
   <!-- Include Utilities -->
-  <xacro:include filename="$(find lbr_iiwa_description)/urdf/utilities.xacro" />
+  <xacro:include filename="$(find yumi_description)/urdf/utilities.xacro" />
   <!-- some constants -->
  <!-- <xacro:property name="safety_controller_k_pos" value="100" />
@@ -12,22 +12,56 @@
   <xacro:property name="joint_damping" value="0.5" />
   <xacro:property name="max_effort" value="300"/>
-  <xacro:property name="max_velocity" value="10"/>
-  <xacro:macro name="lbr_iiwa" params="parent name hardware_interface *origin">
-    <!--joint between {parent} and link_0-->
+  <xacro:macro name="yumi" params="parent name hardware_interface *origin">
+    <!--joint between {parent} and body-->
     <joint name="${parent}_joint" type="fixed">
       <insert_block name="origin"/>
       <parent link="${parent}"/>
-      <child link="${name}_link_0"/>
+      <child link="${name}_body"/>
     </joint>
-    <link name="${name}_link_0">
+    <link name="${name}_body">
       <inertial>
-        <origin xyz="-0.1 0 0.07" rpy="0 0 0"/>
-        <mass value="5"/>
-        <inertia ixx="0.05"  ixy="0"  ixz="0" iyy="0.06" iyz="0" izz="0.03" />
+        <origin xyz="0 0 0" rpy="0 0 0"/>
+        <mass value="15"/>
+        <inertia ixx="0.5"  ixy="0"  ixz="0" iyy="0.6" iyz="0" izz="0.3" />
       </inertial>
       <visual>
         <origin xyz="0 0 0" rpy="0 0 0"/>
         <geometry>
-          <mesh filename="package://lbr_iiwa_description/meshes/link_0.stl"/>
+          <mesh filename="package://yumi_description/meshes/body.stl"/>
+        </geometry>
+        <material name="Light_Grey"/>
+      </visual>
+      <collision>
+        <origin xyz="0 0 0" rpy="0 0 0"/>
+        <geometry>
+          <mesh filename="package://yumi_description/meshes/coarse/body.stl"/>
+        </geometry>
+        <material name="Light_Grey"/>
+      </collision>
+    </link>
+   <!-- joint between body and link_1_r -->
+    <joint name="${name}_joint_1_r" type="revolute">
+      <parent link="${name}_body"/>
+      <child link="${name}_link_1_r"/>
+      <origin xyz="0.05355 -0.0725 0.41492" rpy="-0.9795   -0.5682   -2.3155"/>
+      <axis xyz="0 0 1"/>
+      <limit lower="${-168.5 * PI / 180}" upper="${168.5 * PI / 180}"
+             effort="${max_effort}" velocity="${180 * PI / 180}" />
+      <!--   <safety_controller soft_lower_limit="${-168 * M_PI / 180}"
+           soft_upper_limit="${168 * M_PI / 180}"
+           k_position="${safety_controller_k_pos}"
+           k_velocity="${safety_controller_k_vel}"/> -->
+      <dynamics damping="${joint_damping}"/>
+    </joint>
+   <link name="${name}_link_1_r">
+      <inertial>
+        <origin xyz="0 -0.03 0.12" rpy="0 0 0"/>
+        <mass value="2"/>
+        <inertia ixx="0.1"  ixy="0"  ixz="0" iyy="0.1" iyz="0" izz="0.1" />
+      </inertial>
+      <visual>
+        <origin xyz="0 0 0" rpy="0 0 0"/>
+        <geometry>
+          <mesh filename="package://yumi_description/meshes/link_1.stl"/>
         </geometry>
         <material name="Grey"/>
@@ -36,23 +70,17 @@
         <origin xyz="0 0 0" rpy="0 0 0"/>
         <geometry>
-          <mesh filename="package://lbr_iiwa_description/meshes/coarse/link_0.stl"/>
+          <mesh filename="package://yumi_description/meshes/coarse/link_1.stl"/>
         </geometry>
         <material name="Grey"/>
       </collision>
-      <self_collision_checking>
-        <origin xyz="0 0 0" rpy="0 0 0"/>
-        <geometry>
-          <capsule radius="0.15" length="0.25"/>
-        </geometry>
-      </self_collision_checking>
     </link>
-    <!-- joint between link_0 and link_1 -->
-    <joint name="${name}_joint_1" type="revolute">
-      <parent link="${name}_link_0"/>
-      <child link="${name}_link_1"/>
-      <origin xyz="0 0 0.1575" rpy="0 0 0"/>
+   <!-- joint between link_1_r and link_2_r -->
+    <joint name="${name}_joint_2_r" type="revolute">
+      <parent link="${name}_link_1_r"/>
+      <child link="${name}_link_2_r"/>
+      <origin xyz="0.03 0.0 0.1" rpy="1.5708 0.0 0.0"/>
       <axis xyz="0 0 1"/>
-      <limit lower="${-170 * PI / 180}" upper="${170 * PI / 180}"
-             effort="${max_effort}" velocity="${max_velocity}" />
+      <limit lower="${-143.5 * PI / 180}" upper="${43.5 * PI / 180}"
+             effort="${max_effort}" velocity="${180 * PI / 180}" />
       <!--   <safety_controller soft_lower_limit="${-168 * M_PI / 180}"
            soft_upper_limit="${168 * M_PI / 180}"
@@ -61,224 +89,14 @@
       <dynamics damping="${joint_damping}"/>
     </joint>
-    <link name="${name}_link_1">
+   <link name="${name}_link_2_r">
       <inertial>
-        <origin xyz="0 -0.03 0.12" rpy="0 0 0"/>
-        <mass value="4"/>
-        <inertia ixx="0.1"  ixy="0"  ixz="0" iyy="0.09" iyz="0" izz="0.02" />
+        <origin xyz="0 0 0" rpy="0 0 0"/>
+        <mass value="2"/>
+        <inertia ixx="0.1"  ixy="0"  ixz="0" iyy="0.1" iyz="0" izz="0.1" />
       </inertial>
       <visual>
         <origin xyz="0 0 0" rpy="0 0 0"/>
         <geometry>
-          <mesh filename="package://lbr_iiwa_description/meshes/link_1.stl"/>
-        </geometry>
-        <material name="Orange"/>
-      </visual>
-      <collision>
-        <origin xyz="0 0 0" rpy="0 0 0"/>
-        <geometry>
-          <mesh filename="package://lbr_iiwa_description/meshes/coarse/link_1.stl"/>
-        </geometry>
-        <material name="Orange"/>
-      </collision>
-    </link>
-    <!-- joint between link_1 and link_2 -->
-    <joint name="${name}_joint_2" type="revolute">
-      <parent link="${name}_link_1"/>
-      <child link="${name}_link_2"/>
-      <origin xyz="0 0 0.2025" rpy="${PI / 2}   0 ${PI}"/>
-      <axis xyz="0 0 1"/>
-      <limit lower="${-120 * PI / 180}" upper="${120 * PI / 180}"
-             effort="${max_effort}" velocity="${max_velocity}" />
-      <!-- <safety_controller soft_lower_limit="${-118 * PI / 180}"
-           soft_upper_limit="${118 * PI / 180}"
-           k_position="${safety_controller_k_pos}"
-           k_velocity="${safety_controller_k_vel}"/> -->
-      <dynamics damping="${joint_damping}"/>
-    </joint>
-    <link name="${name}_link_2">
-      <inertial>
-        <origin xyz="0.0003 0.059 0.042" rpy="0 0 0"/>
-        <mass value="4"/>
-        <inertia ixx="0.05"  ixy="0"  ixz="0" iyy="0.018" iyz="0" izz="0.044" />
-      </inertial>
-      <visual>
-        <origin xyz="0 0 0" rpy="0 0 0"/>
-        <geometry>
-          <mesh filename="package://lbr_iiwa_description/meshes/link_2.stl"/>
-        </geometry>
-        <material name="Orange"/>
-      </visual>
-      <collision>
-        <origin xyz="0 0 0" rpy="0 0 0"/>
-        <geometry>
-          <mesh filename="package://lbr_iiwa_description/meshes/coarse/link_2.stl"/>
-        </geometry>
-        <material name="Orange"/>
-      </collision>
-    </link>
-    <!-- joint between link_2 and link_3 -->
-    <joint name="${name}_joint_3" type="revolute">
-      <parent link="${name}_link_2"/>
-      <child link="${name}_link_3"/>
-      <origin xyz="0 0.2045 0" rpy="${PI / 2} 0 ${PI}"/>
-      <axis xyz="0 0 1"/>
-      <limit lower="${-170 * PI / 180}" upper="${170 * PI / 180}"
-             effort="${max_effort}" velocity="${max_velocity}" />
-      <!-- <safety_controller soft_lower_limit="${-118 * PI / 180}"
-           soft_upper_limit="${118 * PI / 180}"
-           k_position="${safety_controller_k_pos}"
-           k_velocity="${safety_controller_k_vel}"/> -->
-      <dynamics damping="${joint_damping}"/>
-    </joint>
-    <link name="${name}_link_3">
-      <inertial>
-        <origin xyz="0 0.03 0.13" rpy="0 0 0"/>
-        <mass value="3"/>
-        <inertia ixx="0.08"  ixy="0"  ixz="0" iyy="0.075" iyz="0" izz="0.01" />
-      </inertial>
-      <visual>
-        <origin xyz="0 0 0" rpy="0 0 0"/>
-        <geometry>
-          <mesh filename="package://lbr_iiwa_description/meshes/link_3.stl"/>
-        </geometry>
-        <material name="Orange"/>
-      </visual>
-      <collision>
-        <origin xyz="0 0 0" rpy="0 0 0"/>
-        <geometry>
-          <mesh filename="package://lbr_iiwa_description/meshes/coarse/link_3.stl"/>
-        </geometry>
-        <material name="Orange"/>
-      </collision>
-    </link>
-   <!-- joint between link_3 and link_4 -->
-    <joint name="${name}_joint_4" type="revolute">
-      <parent link="${name}_link_3"/>
-      <child link="${name}_link_4"/>
-      <origin xyz="0 0 0.2155" rpy="${PI / 2} 0 0"/>
-      <axis xyz="0 0 1"/>
-      <limit lower="${-120 * PI / 180}" upper="${120 * PI / 180}"
-             effort="${max_effort}" velocity="${max_velocity}" />
-      <!-- <safety_controller soft_lower_limit="${-118 * PI / 180}"
-           soft_upper_limit="${118 * PI / 180}"
-           k_position="${safety_controller_k_pos}"
-           k_velocity="${safety_controller_k_vel}"/> -->
-      <dynamics damping="${joint_damping}"/>
-    </joint>
-    <link name="${name}_link_4">
-      <inertial>
-        <origin xyz="0 0.067 0.034" rpy="0 0 0"/>
-        <mass value="2.7"/>
-        <inertia ixx="0.03"  ixy="0"  ixz="0" iyy="0.01" iyz="0" izz="0.029" />
-      </inertial>
-      <visual>
-        <origin xyz="0 0 0" rpy="0 0 0"/>
-        <geometry>
-          <mesh filename="package://lbr_iiwa_description/meshes/link_4.stl"/>
-        </geometry>
-        <material name="Orange"/>
-      </visual>
-      <collision>
-        <origin xyz="0 0 0" rpy="0 0 0"/>
-        <geometry>
-          <mesh filename="package://lbr_iiwa_description/meshes/coarse/link_4.stl"/>
-        </geometry>
-        <material name="Orange"/>
-      </collision>
-    </link>
-    <!-- joint between link_4 and link_5 -->
-    <joint name="${name}_joint_5" type="revolute">
-      <parent link="${name}_link_4"/>
-      <child link="${name}_link_5"/>
-      <origin xyz="0 0.1845 0" rpy="${-PI / 2} ${PI} 0"/>
-      <axis xyz="0 0 1"/>
-      <limit lower="${-170 * PI / 180}" upper="${170 * PI / 180}"
-             effort="${max_effort}" velocity="${max_velocity}" />
-      <!-- <safety_controller soft_lower_limit="${-118 * PI / 180}"
-           soft_upper_limit="${118 * PI / 180}"
-           k_position="${safety_controller_k_pos}"
-           k_velocity="${safety_controller_k_vel}"/> -->
-      <dynamics damping="${joint_damping}"/>
-    </joint>
-    <link name="${name}_link_5">
-      <inertial>
-        <origin xyz="0.0001 0.021 0.076" rpy="0 0 0"/>
-        <mass value="1.7"/>
-        <inertia ixx="0.02"  ixy="0"  ixz="0" iyy="0.018" iyz="0" izz="0.005" />
-      </inertial>
-      <visual>
-        <origin xyz="0 0 0" rpy="0 0 0"/>
-        <geometry>
-          <mesh filename="package://lbr_iiwa_description/meshes/link_5.stl"/>
-        </geometry>
-        <material name="Orange"/>
-      </visual>
-      <collision>
-        <origin xyz="0 0 0" rpy="0 0 0"/>
-        <geometry>
-          <mesh filename="package://lbr_iiwa_description/meshes/coarse/link_5.stl"/>
-        </geometry>
-        <material name="Orange"/>
-      </collision>
-    </link>
- <!-- joint between link_5 and link_6 -->
-    <joint name="${name}_joint_6" type="revolute">
-      <parent link="${name}_link_5"/>
-      <child link="${name}_link_6"/>
-      <origin xyz="0 0 0.2155" rpy="${PI / 2} 0 0"/>
-      <axis xyz="0 0 1"/>
-      <limit lower="${-120 * PI / 180}" upper="${120 * PI / 180}"
-             effort="${max_effort}" velocity="${max_velocity}" />
-      <!-- <safety_controller soft_lower_limit="${-118 * PI / 180}"
-           soft_upper_limit="${118 * PI / 180}"
-           k_position="${safety_controller_k_pos}"
-           k_velocity="${safety_controller_k_vel}"/> -->
-      <dynamics damping="${joint_damping}"/>
-    </joint>
-    <link name="${name}_link_6">
-      <inertial>
-        <origin xyz="0 0.0006 0.0004" rpy="0 0 0"/>
-        <mass value="1.8"/>
-        <inertia ixx="0.005"  ixy="0"  ixz="0" iyy="0.0036" iyz="0" izz="0.0047" />
-      </inertial>
-      <visual>
-        <origin xyz="0 0 0" rpy="0 0 0"/>
-        <geometry>
-          <mesh filename="package://lbr_iiwa_description/meshes/link_6.stl"/>
-        </geometry>
-        <material name="Orange"/>
-      </visual>
-      <collision>
-        <origin xyz="0 0 0" rpy="0 0 0"/>
-        <geometry>
-          <mesh filename="package://lbr_iiwa_description/meshes/coarse/link_6.stl"/>
-        </geometry>
-        <material name="Orange"/>
-      </collision>
-    </link>
- <!-- joint between link_6 and link_7 -->
-    <joint name="${name}_joint_7" type="revolute">
-      <parent link="${name}_link_6"/>
-      <child link="${name}_link_7"/>
-      <origin xyz="0 0.081 0" rpy="${- PI / 2} ${PI} 0"/>
-      <axis xyz="0 0 1"/>
-      <limit lower="${-175 * PI / 180}" upper="${175 * PI / 180}"
-             effort="${max_effort}" velocity="${max_velocity}" />
-      <!-- <safety_controller soft_lower_limit="${-118 * PI / 180}"
-           soft_upper_limit="${118 * PI / 180}"
-           k_position="${safety_controller_k_pos}"
-           k_velocity="${safety_controller_k_vel}"/> -->
-      <dynamics damping="${joint_damping}"/>
-    </joint>
-    <link name="${name}_link_7">
-      <inertial>
-        <origin xyz="0 0 0.02" rpy="0 0 0"/>
-        <mass value="0.3"/>
-        <inertia ixx="0.001"  ixy="0"  ixz="0" iyy="0.001" iyz="0" izz="0.001" />
-      </inertial>
-      <visual>
-        <origin xyz="0 0 0" rpy="0 0 0"/>
-        <geometry>
-          <mesh filename="package://lbr_iiwa_description/meshes/link_7.stl"/>
+          <mesh filename="package://yumi_description/meshes/link_2.stl"/>
         </geometry>
         <material name="Grey"/>
@@ -287,5 +105,75 @@
         <origin xyz="0 0 0" rpy="0 0 0"/>
         <geometry>
-          <mesh filename="package://lbr_iiwa_description/meshes/coarse/link_7.stl"/>
+          <mesh filename="package://yumi_description/meshes/coarse/link_2.stl"/>
+        </geometry>
+        <material name="Grey"/>
+      </collision>
+    </link>
+   <!-- joint between link_2_r and link_3_r -->
+    <joint name="${name}_joint_3_r" type="revolute">
+      <parent link="${name}_link_2_r"/>
+      <child link="${name}_link_3_r"/>
+      <origin xyz="-0.03 0.17283 0.0" rpy="-1.5708 0.0 0.0"/>
+      <axis xyz="0 0 1"/>
+      <limit lower="${-168.5 * PI / 180}" upper="${168.5 * PI / 180}"
+             effort="${max_effort}" velocity="${180 * PI / 180}" />
+      <!--   <safety_controller soft_lower_limit="${-168 * M_PI / 180}"
+           soft_upper_limit="${168 * M_PI / 180}"
+           k_position="${safety_controller_k_pos}"
+           k_velocity="${safety_controller_k_vel}"/> -->
+      <dynamics damping="${joint_damping}"/>
+    </joint>
+   <link name="${name}_link_3_r">
+      <inertial>
+        <origin xyz="0 0 0" rpy="0 0 0"/>
+        <mass value="2"/>
+        <inertia ixx="0.1"  ixy="0"  ixz="0" iyy="0.1" iyz="0" izz="0.1" />
+      </inertial>
+      <visual>
+        <origin xyz="0 0 0" rpy="0 0 0"/>
+        <geometry>
+          <mesh filename="package://yumi_description/meshes/link_3.stl"/>
+        </geometry>
+        <material name="Grey"/>
+      </visual>
+      <collision>
+        <origin xyz="0 0 0" rpy="0 0 0"/>
+        <geometry>
+          <mesh filename="package://yumi_description/meshes/coarse/link_3.stl"/>
+        </geometry>
+        <material name="Grey"/>
+      </collision>
+    </link>
+   <!-- joint between link_3_r and link_4_r -->
+    <joint name="${name}_joint_4_r" type="revolute">
+      <parent link="${name}_link_3_r"/>
+      <child link="${name}_link_4_r"/>
+      <origin xyz="-0.04188 0.0 0.07873" rpy="1.5708 -1.5708 0.0"/>
+      <axis xyz="0 0 1"/>
+      <limit lower="${-123.5 * PI / 180}" upper="${80 * PI / 180}"
+             effort="${max_effort}" velocity="${180 * PI / 180}" />
+      <!--   <safety_controller soft_lower_limit="${-168 * M_PI / 180}"
+           soft_upper_limit="${168 * M_PI / 180}"
+           k_position="${safety_controller_k_pos}"
+           k_velocity="${safety_controller_k_vel}"/> -->
+      <dynamics damping="${joint_damping}"/>
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