Commit message: Updated YuMi URDF/XACRO files
Remove unnecessary XACRO files, and create new files in order to generate the proper YuMi URDF file

File: yumi_description/urdf/materials.xacro (robot description, xacro)
@@ -1,3 +1,10 @@
 <?xml version="1.0"?>
+<!--
+  PROGRAMMER: Frederick Wachter
+  DATE CREATED: 2016-05-30
+  LAST MODIFIED: 2016-05-30
+  PURPOSE: Provide colors for the different objects in the YuMi workspace
+  REFERENCE: https://github.com/rtkg/yumi
+-->
 <robot>
   <material name="Black">
@@ -31,3 +38,12 @@
     <color rgba="1.0 1.0 1.0 1.0"/>
   </material>
+  <material name="Drexel_Blue">
+    <color rgba="0.027 0.161 0.302 1.0"/>
+  </material>
+  <material name="SeeThrough">
+    <color rgba="0 0 0 0"/>
+  </material>
+  <material name="Transparent">
+    <color rgba="1.0 1.0 1.0 0.5"/>
+  </material>
 </robot>

File: yumi_description/urdf/utilities.xacro (robot description, xacro)
@@ -1,20 +1,14 @@
 <?xml version="1.0"?>
-<robot name="lbr_iiwa" xmlns:xacro="http://www.ros.org/wiki/xacro">
+<!--
+  PROGRAMMER: Frederick Wachter
+  DATE CREATED: 2016-05-30
+  LAST MODIFIED: 2016-05-30
+  PURPOSE: Provide constants and modeling macros for YuMi
+  REFERENCE: https://github.com/rtkg/yumi
+-->
+<robot name="yumi" xmlns:xacro="http://www.ros.org/wiki/xacro">
+  <!-- Constants -->
   <xacro:property name="PI" value="3.1415926535897931"/>
-<!-- The following macros are adapted from the LWR 4 definitions of the RCPRG - https://github.com/RCPRG-ros-pkg/lwr_robot -->
-  <!--Little helper macros to define the inertia matrix needed for links.-->
-  <!--Cuboid-->
-  <xacro:macro name="cuboid_inertia" params="width height length mass">
-    <inertia ixx="${mass * (height * height + length * length) / 12)}"
-             iyy="${mass * (width * width + length * length) / 12)}"
-             izz="${mass * (width * width + height * height) / 12)}"
-             ixy="0" iyz="0" ixz="0"/>
-  </xacro:macro>
-  <!--Cylinder: length is along the y-axis! -->
-  <xacro:macro name="cylinder_inertia" params="radius length mass">
-    <inertia ixx="${mass * (3 * radius * radius + length * length) / 12)}"
-             iyy="${mass * radius* radius / 2)}"
-             izz="${mass * (3 * radius * radius + length * length) / 12)}"
-             ixy="0" iyz="0" ixz="0"/>
-  </xacro:macro>
+  <!-- Model Properties -->
+  <xacro:property name="hardware_interface" value="yumi"/>
 </robot>

File: yumi_description/urdf/yumi.transmission.xacro (robot description, xacro)
@@ -1,3 +1,10 @@
 <?xml version="1.0"?>
+<!--
+  PROGRAMMER: Frederick Wachter
+  DATE CREATED: 2016-05-30
+  LAST MODIFIED: 2016-05-30
+  PURPOSE: Provide colors for the different objects in the YuMi workspace
+  REFERENCE: https://github.com/rtkg/yumi
+-->
 <robot name="yumi" xmlns:xacro="http://www.ros.org/wiki/xacro">
   <xacro:macro name="yumi_transmission" params="name hardware_interface">
@@ -5,9 +12,9 @@
       <type>transmission_interface/SimpleTransmission</type>
       <joint name="${name}_joint_1_r">
-	<hardwareInterface>${hardware_interface}</hardwareInterface>
+        <hardwareInterface>${hardware_interface}</hardwareInterface>
       </joint>
       <actuator name="${name}_motor_1_r">
-	<hardwareInterface>${hardware_interface}</hardwareInterface>
-	<mechanicalReduction>1</mechanicalReduction>
+        <hardwareInterface>${hardware_interface}</hardwareInterface>
+        <mechanicalReduction>1</mechanicalReduction>
       </actuator>
     </transmission>
@@ -15,9 +22,9 @@
       <type>transmission_interface/SimpleTransmission</type>
       <joint name="${name}_joint_2_r">
-	<hardwareInterface>${hardware_interface}</hardwareInterface>
+        <hardwareInterface>${hardware_interface}</hardwareInterface>
       </joint>
       <actuator name="${name}_motor_2_r">
-	<hardwareInterface>${hardware_interface}</hardwareInterface>
-	<mechanicalReduction>1</mechanicalReduction>
+        <hardwareInterface>${hardware_interface}</hardwareInterface>
+        <mechanicalReduction>1</mechanicalReduction>
       </actuator>
     </transmission>
@@ -25,9 +32,9 @@
       <type>transmission_interface/SimpleTransmission</type>
       <joint name="${name}_joint_3_r">
-	<hardwareInterface>${hardware_interface}</hardwareInterface>
+        <hardwareInterface>${hardware_interface}</hardwareInterface>
       </joint>
       <actuator name="${name}_motor_3_r">
-	<hardwareInterface>${hardware_interface}</hardwareInterface>
-	<mechanicalReduction>1</mechanicalReduction>
+        <hardwareInterface>${hardware_interface}</hardwareInterface>
+        <mechanicalReduction>1</mechanicalReduction>
       </actuator>
     </transmission>
@@ -35,9 +42,9 @@
       <type>transmission_interface/SimpleTransmission</type>
       <joint name="${name}_joint_4_r">
-	<hardwareInterface>${hardware_interface}</hardwareInterface>
+        <hardwareInterface>${hardware_interface}</hardwareInterface>
       </joint>
       <actuator name="${name}_motor_4_r">
-	<hardwareInterface>${hardware_interface}</hardwareInterface>
-	<mechanicalReduction>1</mechanicalReduction>
+        <hardwareInterface>${hardware_interface}</hardwareInterface>
+        <mechanicalReduction>1</mechanicalReduction>
       </actuator>
     </transmission>
@@ -45,9 +52,9 @@
       <type>transmission_interface/SimpleTransmission</type>
       <joint name="${name}_joint_5_r">
-	<hardwareInterface>${hardware_interface}</hardwareInterface>
+        <hardwareInterface>${hardware_interface}</hardwareInterface>
       </joint>
       <actuator name="${name}_motor_5_r">
-	<hardwareInterface>${hardware_interface}</hardwareInterface>
-	<mechanicalReduction>1</mechanicalReduction>
+        <hardwareInterface>${hardware_interface}</hardwareInterface>
+        <mechanicalReduction>1</mechanicalReduction>
       </actuator>
     </transmission>
@@ -55,9 +62,9 @@
       <type>transmission_interface/SimpleTransmission</type>
       <joint name="${name}_joint_6_r">
-	<hardwareInterface>${hardware_interface}</hardwareInterface>
+        <hardwareInterface>${hardware_interface}</hardwareInterface>
       </joint>
       <actuator name="${name}_motor_6_r">
-	<hardwareInterface>${hardware_interface}</hardwareInterface>
-	<mechanicalReduction>1</mechanicalReduction>
+        <hardwareInterface>${hardware_interface}</hardwareInterface>
+        <mechanicalReduction>1</mechanicalReduction>
       </actuator>
     </transmission>
@@ -65,9 +72,9 @@
       <type>transmission_interface/SimpleTransmission</type>
       <joint name="${name}_joint_7_r">
-	<hardwareInterface>${hardware_interface}</hardwareInterface>
+        <hardwareInterface>${hardware_interface}</hardwareInterface>
       </joint>
       <actuator name="${name}_motor_7_r">
-	<hardwareInterface>${hardware_interface}</hardwareInterface>
-	<mechanicalReduction>1</mechanicalReduction>
+        <hardwareInterface>${hardware_interface}</hardwareInterface>
+        <mechanicalReduction>1</mechanicalReduction>
       </actuator>
     </transmission>
@@ -75,9 +82,9 @@
       <type>transmission_interface/SimpleTransmission</type>
       <joint name="${name}_joint_1_l">
-	<hardwareInterface>${hardware_interface}</hardwareInterface>
+        <hardwareInterface>${hardware_interface}</hardwareInterface>
       </joint>
       <actuator name="${name}_motor_1_l">
-	<hardwareInterface>${hardware_interface}</hardwareInterface>
-	<mechanicalReduction>1</mechanicalReduction>
+        <hardwareInterface>${hardware_interface}</hardwareInterface>
+        <mechanicalReduction>1</mechanicalReduction>
       </actuator>
     </transmission>
@@ -85,9 +92,9 @@
       <type>transmission_interface/SimpleTransmission</type>
       <joint name="${name}_joint_2_l">
-	<hardwareInterface>${hardware_interface}</hardwareInterface>
+        <hardwareInterface>${hardware_interface}</hardwareInterface>
       </joint>
       <actuator name="${name}_motor_2_l">
-	<hardwareInterface>${hardware_interface}</hardwareInterface>
-	<mechanicalReduction>1</mechanicalReduction>
+        <hardwareInterface>${hardware_interface}</hardwareInterface>
+        <mechanicalReduction>1</mechanicalReduction>
       </actuator>
     </transmission>
@@ -95,9 +102,9 @@
       <type>transmission_interface/SimpleTransmission</type>
       <joint name="${name}_joint_3_l">
-	<hardwareInterface>${hardware_interface}</hardwareInterface>
+        <hardwareInterface>${hardware_interface}</hardwareInterface>
       </joint>
       <actuator name="${name}_motor_3_l">
-	<hardwareInterface>${hardware_interface}</hardwareInterface>
-	<mechanicalReduction>1</mechanicalReduction>
+        <hardwareInterface>${hardware_interface}</hardwareInterface>
+        <mechanicalReduction>1</mechanicalReduction>
       </actuator>
     </transmission>
@@ -105,9 +112,9 @@
       <type>transmission_interface/SimpleTransmission</type>
       <joint name="${name}_joint_4_l">
-	<hardwareInterface>${hardware_interface}</hardwareInterface>
+        <hardwareInterface>${hardware_interface}</hardwareInterface>
       </joint>
       <actuator name="${name}_motor_4_l">
-	<hardwareInterface>${hardware_interface}</hardwareInterface>
-	<mechanicalReduction>1</mechanicalReduction>
+        <hardwareInterface>${hardware_interface}</hardwareInterface>
+        <mechanicalReduction>1</mechanicalReduction>
       </actuator>
     </transmission>
@@ -115,9 +122,9 @@
       <type>transmission_interface/SimpleTransmission</type>
       <joint name="${name}_joint_5_l">
-	<hardwareInterface>${hardware_interface}</hardwareInterface>
+        <hardwareInterface>${hardware_interface}</hardwareInterface>
       </joint>
       <actuator name="${name}_motor_5_l">
-	<hardwareInterface>${hardware_interface}</hardwareInterface>
-	<mechanicalReduction>1</mechanicalReduction>
+        <hardwareInterface>${hardware_interface}</hardwareInterface>
+        <mechanicalReduction>1</mechanicalReduction>
       </actuator>
     </transmission>
@@ -125,9 +132,9 @@
       <type>transmission_interface/SimpleTransmission</type>
       <joint name="${name}_joint_6_l">
-	<hardwareInterface>${hardware_interface}</hardwareInterface>
+        <hardwareInterface>${hardware_interface}</hardwareInterface>
       </joint>
       <actuator name="${name}_motor_6_l">
-	<hardwareInterface>${hardware_interface}</hardwareInterface>
-	<mechanicalReduction>1</mechanicalReduction>
+        <hardwareInterface>${hardware_interface}</hardwareInterface>
+        <mechanicalReduction>1</mechanicalReduction>
       </actuator>
     </transmission>
@@ -135,9 +142,9 @@
       <type>transmission_interface/SimpleTransmission</type>
       <joint name="${name}_joint_7_l">
-	<hardwareInterface>${hardware_interface}</hardwareInterface>
+        <hardwareInterface>${hardware_interface}</hardwareInterface>
       </joint>
       <actuator name="${name}_motor_7_l">
-	<hardwareInterface>${hardware_interface}</hardwareInterface>
-	<mechanicalReduction>1</mechanicalReduction>
+        <hardwareInterface>${hardware_interface}</hardwareInterface>
+        <mechanicalReduction>1</mechanicalReduction>
       </actuator>
     </transmission>

File: yumi_description/urdf/yumi.urdf (robot description, URDF)
Before this commit: robot yumi, 27 links, 26 joints
Joints:
- removed joint tableTop_to_table
- added joint table_top_to_table: type fixed, parent table, child table_top, origin xyz=0 0 0 rpy=0 0 0
- joint base_to_stand: origin xyz=165.50539 0.00284 0.10014 rpy=0 0 0 -> xyz=0 0 0 rpy=0 0 0
- joint stand_to_world: origin xyz=-0.466 -0.26 0 rpy=0 0 0 -> xyz=0 0 0 rpy=0 0 0; parent world -> yumi_body

File: yumi_description/urdf/yumi.urdf.xacro (robot description, xacro)
@@ -1,27 +1,46 @@
 <?xml version="1.0"?>
+<!--
+  PROGRAMMER: Frederick Wachter
+  DATE CREATED: 2016-05-30
+  LAST MODIFIED: 2016-05-30
+  PURPOSE: Import necessary files to build YuMi URDF with workspace
+-->
 <robot name="yumi" xmlns:xacro="http://www.ros.org/wiki/xacro">
-  <!-- Import Rviz colors -->
-  <xacro:include filename="$(find yumi_description)/urdf/materials.xacro" />
-  <!-- Import utilities -->
-  <xacro:include filename="$(find yumi_description)/urdf/utilities.xacro" />
-  <!--Import the yumi macro -->
+  <!--                  		   -->
+  <!--         IMPORTS         -->
+  <!--                  		   -->
+  <!-- Import Colors -->
+  <xacro:include filename="$(find yumi_description)/urdf/materials.xacro"/>
+  <!-- Import Constants and Modeling Macros -->
+  <xacro:include filename="$(find yumi_description)/urdf/utilities.xacro"/>
+  <!-- Import Workspace -->
+  <xacro:include filename="$(find yumi_description)/urdf/workspace.xacro"/>
+  <!-- Import YuMi -->
   <xacro:include filename="$(find yumi_description)/urdf/yumi.xacro"/>
-  <!--Import the yumi servo gripper macro -->
+  <!-- Import Right Servo Gripper -->
   <xacro:include filename="$(find yumi_description)/urdf/yumi_servo_gripper.xacro"/>
- <!-- Import Gazebo plugins -->
-  <xacro:include filename="$(find yumi_description)/gazebo/gazebo.urdf.xacro"/>
-  <!-- Fix to world just for testing -->
+  <!-- Import Camera Assembly -->
+  <xacro:include filename="$(find yumi_description)/urdf/camera_assembly.xacro"/>
+  <!--                  		   -->
+  <!--     LINK DEFINITIONS    -->
+  <!--                  		   -->
+  <!-- World Fixed Link for YuMi -->
   <link name="world"/>
-  <!--yumi-->
-  <xacro:yumi name="yumi" hardware_interface="$(arg prefix)" parent="world">
-    <origin xyz="0 0 0.1" rpy="0 0 0" />
+  <!--                  		   -->
+  <!--    MACRO DEFINITIONS    -->
+  <!--                  		   -->
+  <!-- Define Macros for YuMi Import -->
+  <xacro:yumi name="yumi" hardware_interface="${hardware_interface}" parent="world">
+	  <origin xyz="0 0 0.1" rpy="0 0 0"/> <!-- Bring bottom of YuMi to (x,y) plane -->
   </xacro:yumi>
-  <!--right gripper-->
-  <xacro:yumi_servo_gripper name="gripper_r" hardware_interface="$(arg prefix)" parent="yumi_link_7_r">
-    <origin xyz="0 0 0.007" rpy="0 0 ${PI}" />
+  <!-- Define Macros for Workspace Import -->
+  <xacro:workspace stand_parent="yumi_body" table_parent="world">
+    <origin rpy="0 0 0" xyz="-0.07 0.54 -0.013"/>
+  </xacro:workspace>
+  <!-- Define Macros for Right Servo Gripper Import -->
+  <xacro:yumi_servo_gripper name="gripper_r" hardware_interface="${hardware_interface}" parent="yumi_link_7_r">
+  	<origin xyz="0 0 0.007" rpy="0 0 ${PI}"/>
   </xacro:yumi_servo_gripper>
-  <!--left gripper-->
-  <xacro:yumi_servo_gripper name="gripper_l" hardware_interface="$(arg prefix)" parent="yumi_link_7_l">
-    <origin xyz="0 0 0.007" rpy="0 0 ${PI}" />
-  </xacro:yumi_servo_gripper>
+  <!-- Define Macros for Camera Assembly Import -->
+  <xacro:camera_assembly parent="yumi_link_7_l"/>
 </robot>
