Commit message: Updated YuMi URDF/XACRO files
Remove unnecessary XACRO files, and create new files in order to generate the proper YuMi URDF file

File: yumi_description/urdf/yumi.xacro (robot description, xacro)
@@ -1,17 +1,22 @@
 <?xml version="1.0"?>
+<!--
+  PROGRAMMER: Frederick Wachter
+  DATE CREATED: 2016-05-30
+  LAST MODIFIED: 2016-05-30
+  PURPOSE: Provide colors for the different objects in the YuMi workspace
+  REFERENCE: https://github.com/rtkg/yumi
+-->
 <robot name="yumi" xmlns:xacro="http://www.ros.org/wiki/xacro">
-  <!-- Import all Gazebo-customization elements, including Gazebo colors -->
-  <xacro:include filename="$(find yumi_description)/urdf/yumi.gazebo.xacro" />
   <!-- Import Transmissions -->
   <xacro:include filename="$(find yumi_description)/urdf/yumi.transmission.xacro" />
   <!-- Include Utilities -->
   <xacro:include filename="$(find yumi_description)/urdf/utilities.xacro" />
-  <!-- some constants -->
- <!-- <xacro:property name="safety_controller_k_pos" value="100" />
-  <xacro:property name="safety_controller_k_vel" value="2" /> -->
+  <!-- Constants -->
   <xacro:property name="joint_damping" value="0.5" />
   <xacro:property name="max_effort" value="300"/>
   <xacro:macro name="yumi" params="parent name hardware_interface *origin">
-    <!--joint between {parent} and body-->
+    <!--                         -->
+    <!--           BODY          -->
+    <!--                         -->
     <joint name="${parent}_joint" type="fixed">
       <insert_block name="origin"/>
@@ -40,6 +45,7 @@
       </collision>
     </link>
-   <!--///////////////////////////////////// RIGHT ARM ////////////////////////////////  -->
-   <!-- joint between body and link_1_r -->
+    <!--                         -->
+    <!--        RIGHT ARM        -->
+    <!--                         -->
     <joint name="${name}_joint_1_r" type="revolute">
       <parent link="${name}_body"/>
@@ -47,13 +53,8 @@
       <origin xyz="0.05355 -0.0725 0.41492" rpy="-0.9795   -0.5682   -2.3155"/>
       <axis xyz="0 0 1"/>
-      <limit lower="${-168.5 * PI / 180}" upper="${168.5 * PI / 180}"
-             effort="${max_effort}" velocity="${180 * PI / 180}" />
-      <!--   <safety_controller soft_lower_limit="${-168 * M_PI / 180}"
-           soft_upper_limit="${168 * M_PI / 180}"
-           k_position="${safety_controller_k_pos}"
-           k_velocity="${safety_controller_k_vel}"/> -->
-      <dynamics damping="${joint_damping}"/>
-    </joint>
-   <link name="${name}_link_1_r">
+      <limit lower="${-168.5 * PI / 180}" upper="${168.5 * PI / 180}" effort="${max_effort}" velocity="${180 * PI / 180}" />
+      <dynamics damping="${joint_damping}"/>
+    </joint>
+    <link name="${name}_link_1_r">
       <inertial>
         <origin xyz="0 -0.03 0.12" rpy="0 0 0"/>
@@ -76,5 +77,4 @@
       </collision>
     </link>
-   <!-- joint between link_1_r and link_2_r -->
     <joint name="${name}_joint_2_r" type="revolute">
       <parent link="${name}_link_1_r"/>
@@ -82,13 +82,8 @@
       <origin xyz="0.03 0.0 0.1" rpy="${PI / 2} 0.0 0.0"/>
       <axis xyz="0 0 1"/>
-      <limit lower="${-143.5 * PI / 180}" upper="${43.5 * PI / 180}"
-             effort="${max_effort}" velocity="${180 * PI / 180}" />
-      <!--   <safety_controller soft_lower_limit="${-168 * M_PI / 180}"
-           soft_upper_limit="${168 * M_PI / 180}"
-           k_position="${safety_controller_k_pos}"
-           k_velocity="${safety_controller_k_vel}"/> -->
-      <dynamics damping="${joint_damping}"/>
-    </joint>
-   <link name="${name}_link_2_r">
+      <limit lower="${-143.5 * PI / 180}" upper="${43.5 * PI / 180}" effort="${max_effort}" velocity="${180 * PI / 180}" />
+      <dynamics damping="${joint_damping}"/>
+    </joint>
+    <link name="${name}_link_2_r">
       <inertial>
         <origin xyz="0 0 0" rpy="0 0 0"/>
@@ -111,5 +106,4 @@
       </collision>
     </link>
-   <!-- joint between link_2_r and link_3_r -->
     <joint name="${name}_joint_7_r" type="revolute">
       <parent link="${name}_link_2_r"/>
@@ -117,13 +111,8 @@
       <origin xyz="-0.03 0.17283 0.0" rpy="${-PI / 2} 0.0 0.0"/>
       <axis xyz="0 0 1"/>
-      <limit lower="${-168.5 * PI / 180}" upper="${168.5 * PI / 180}"
-             effort="${max_effort}" velocity="${180 * PI / 180}" />
-      <!--   <safety_controller soft_lower_limit="${-168 * M_PI / 180}"
-           soft_upper_limit="${168 * M_PI / 180}"
-           k_position="${safety_controller_k_pos}"
-           k_velocity="${safety_controller_k_vel}"/> -->
-      <dynamics damping="${joint_damping}"/>
-    </joint>
-   <link name="${name}_link_3_r">
+      <limit lower="${-168.5 * PI / 180}" upper="${168.5 * PI / 180}" effort="${max_effort}" velocity="${180 * PI / 180}" />
+      <dynamics damping="${joint_damping}"/>
+    </joint>
+    <link name="${name}_link_3_r">
       <inertial>
         <origin xyz="0 0 0" rpy="0 0 0"/>
@@ -146,5 +135,4 @@
       </collision>
     </link>
-   <!-- joint between link_3_r and link_4_r -->
     <joint name="${name}_joint_3_r" type="revolute">
       <parent link="${name}_link_3_r"/>
@@ -152,13 +140,8 @@
       <origin xyz="-0.04188 0.0 0.07873" rpy="${PI / 2} ${- PI / 2} 0.0"/>
       <axis xyz="0 0 1"/>
-      <limit lower="${-123.5 * PI / 180}" upper="${80 * PI / 180}"
-             effort="${max_effort}" velocity="${180 * PI / 180}" />
-      <!--   <safety_controller soft_lower_limit="${-168 * M_PI / 180}"
-           soft_upper_limit="${168 * M_PI / 180}"
-           k_position="${safety_controller_k_pos}"
-           k_velocity="${safety_controller_k_vel}"/> -->
-      <dynamics damping="${joint_damping}"/>
-    </joint>
-   <link name="${name}_link_4_r">
+      <limit lower="${-123.5 * PI / 180}" upper="${80 * PI / 180}" effort="${max_effort}" velocity="${180 * PI / 180}" />
+      <dynamics damping="${joint_damping}"/>
+    </joint>
+    <link name="${name}_link_4_r">
       <inertial>
         <origin xyz="0 0 0" rpy="0 0 0"/>
@@ -181,5 +164,4 @@
       </collision>
     </link>
-   <!-- joint between link_4_r and link_5_r -->
     <joint name="${name}_joint_4_r" type="revolute">
       <parent link="${name}_link_4_r"/>
@@ -187,13 +169,8 @@
       <origin xyz="0.0405 0.16461 0.0" rpy="-${PI / 2} 0.0 0.0"/>
       <axis xyz="0 0 1"/>
-      <limit lower="${-290 * PI / 180}" upper="${290 * PI / 180}"
-             effort="${max_effort}" velocity="${400 * PI / 180}" />
-      <!--   <safety_controller soft_lower_limit="${-168 * M_PI / 180}"
-           soft_upper_limit="${168 * M_PI / 180}"
-           k_position="${safety_controller_k_pos}"
-           k_velocity="${safety_controller_k_vel}"/> -->
-      <dynamics damping="${joint_damping}"/>
-    </joint>
-   <link name="${name}_link_5_r">
+      <limit lower="${-290 * PI / 180}" upper="${290 * PI / 180}" effort="${max_effort}" velocity="${400 * PI / 180}" />
+      <dynamics damping="${joint_damping}"/>
+    </joint>
+    <link name="${name}_link_5_r">
       <inertial>
         <origin xyz="0 0 0" rpy="0 0 0"/>
@@ -216,5 +193,4 @@
       </collision>
     </link>
-   <!-- joint between link_5_r and link_6_r -->
     <joint name="${name}_joint_5_r" type="revolute">
       <parent link="${name}_link_5_r"/>
@@ -222,13 +198,8 @@
       <origin xyz="-0.027 0 0.10039" rpy="${PI / 2} 0.0 0.0"/>
       <axis xyz="0 0 1"/>
-      <limit lower="${-88 * PI / 180}" upper="${138 * PI / 180}"
-             effort="${max_effort}" velocity="${400 * PI / 180}" />
-      <!--   <safety_controller soft_lower_limit="${-168 * M_PI / 180}"
-           soft_upper_limit="${168 * M_PI / 180}"
-           k_position="${safety_controller_k_pos}"
-           k_velocity="${safety_controller_k_vel}"/> -->
-      <dynamics damping="${joint_damping}"/>
-    </joint>
-   <link name="${name}_link_6_r">
+      <limit lower="${-88 * PI / 180}" upper="${138 * PI / 180}" effort="${max_effort}" velocity="${400 * PI / 180}" />
+      <dynamics damping="${joint_damping}"/>
+    </joint>
+    <link name="${name}_link_6_r">
       <inertial>
         <origin xyz="0 0 0" rpy="0 0 0"/>
@@ -251,5 +222,4 @@
       </collision>
     </link>
-   <!-- joint between link_6_r and link_7_r -->
     <joint name="${name}_joint_6_r" type="revolute">
       <parent link="${name}_link_6_r"/>
@@ -257,13 +227,8 @@
       <origin xyz="0.027 0.029 0.0" rpy="-${PI / 2} 0.0 0.0"/>
       <axis xyz="0 0 1"/>
-      <limit lower="${-229 * PI / 180}" upper="${229 * PI / 180}"
-             effort="${max_effort}" velocity="${400 * PI / 180}" />
-      <!--   <safety_controller soft_lower_limit="${-168 * M_PI / 180}"
-           soft_upper_limit="${168 * M_PI / 180}"
-           k_position="${safety_controller_k_pos}"
-           k_velocity="${safety_controller_k_vel}"/> -->
-      <dynamics damping="${joint_damping}"/>
-    </joint>
-   <link name="${name}_link_7_r">
+      <limit lower="${-229 * PI / 180}" upper="${229 * PI / 180}" effort="${max_effort}" velocity="${400 * PI / 180}" />
+      <dynamics damping="${joint_damping}"/>
+    </joint>
+    <link name="${name}_link_7_r">
       <inertial>
         <origin xyz="0 0 0" rpy="0 0 0"/>
@@ -286,6 +251,7 @@
       </collision>
     </link>
-   <!--///////////////////////////////////// LEFT ARM ////////////////////////////////  -->
-  <!-- joint between body and link_1_l -->
+    <!--                         -->
+    <!--        LEFT ARM         -->
+    <!--                         -->
     <joint name="${name}_joint_1_l" type="revolute">
       <parent link="${name}_body"/>
@@ -293,13 +259,8 @@
       <origin xyz="0.05355 0.07250 0.41492" rpy="0.9781 -0.5716 2.3180"/>
       <axis xyz="0 0 1"/>
-      <limit lower="${-168.5 * PI / 180}" upper="${168.5 * PI / 180}"
-             effort="${max_effort}" velocity="${180 * PI / 180}" />
-      <!--   <safety_controller soft_lower_limit="${-168 * M_PI / 180}"
-           soft_upper_limit="${168 * M_PI / 180}"
-           k_position="${safety_controller_k_pos}"
-           k_velocity="${safety_controller_k_vel}"/> -->
-      <dynamics damping="${joint_damping}"/>
-    </joint>
-   <link name="${name}_link_1_l">
+      <limit lower="${-168.5 * PI / 180}" upper="${168.5 * PI / 180}" effort="${max_effort}" velocity="${180 * PI / 180}" />
+      <dynamics damping="${joint_damping}"/>
+    </joint>
+    <link name="${name}_link_1_l">
       <inertial>
         <origin xyz="0 -0.03 0.12" rpy="0 0 0"/>
@@ -322,5 +283,4 @@
       </collision>
     </link>
- <!-- joint between link_1_l and link_2_l -->
     <joint name="${name}_joint_2_l" type="revolute">
       <parent link="${name}_link_1_l"/>
@@ -328,13 +288,8 @@
       <origin xyz="0.03 0.0 0.1" rpy="${PI / 2} 0.0 0.0"/>
       <axis xyz="0 0 1"/>
-      <limit lower="${-143.5 * PI / 180}" upper="${43.5 * PI / 180}"
-             effort="${max_effort}" velocity="${180 * PI / 180}" />
-      <!--   <safety_controller soft_lower_limit="${-168 * M_PI / 180}"
-           soft_upper_limit="${168 * M_PI / 180}"
-           k_position="${safety_controller_k_pos}"
-           k_velocity="${safety_controller_k_vel}"/> -->
-      <dynamics damping="${joint_damping}"/>
-    </joint>
-   <link name="${name}_link_2_l">
+      <limit lower="${-143.5 * PI / 180}" upper="${43.5 * PI / 180}" effort="${max_effort}" velocity="${180 * PI / 180}" />
+      <dynamics damping="${joint_damping}"/>
+    </joint>
+    <link name="${name}_link_2_l">
       <inertial>
         <origin xyz="0 0 0" rpy="0 0 0"/>
@@ -357,5 +312,4 @@
       </collision>
     </link>
- <!-- joint between link_2_l and link_3_l -->
     <joint name="${name}_joint_7_l" type="revolute">
       <parent link="${name}_link_2_l"/>
@@ -363,13 +317,8 @@
       <origin xyz="-0.03 0.17283 0.0" rpy="-${PI / 2} 0.0 0.0"/>
       <axis xyz="0 0 1"/>
-      <limit lower="${-168.5 * PI / 180}" upper="${168.5 * PI / 180}"
-             effort="${max_effort}" velocity="${180 * PI / 180}" />
-      <!--   <safety_controller soft_lower_limit="${-168 * M_PI / 180}"
-           soft_upper_limit="${168 * M_PI / 180}"
-           k_position="${safety_controller_k_pos}"
-           k_velocity="${safety_controller_k_vel}"/> -->
-      <dynamics damping="${joint_damping}"/>
-    </joint>
-   <link name="${name}_link_3_l">
+      <limit lower="${-168.5 * PI / 180}" upper="${168.5 * PI / 180}" effort="${max_effort}" velocity="${180 * PI / 180}" />
+      <dynamics damping="${joint_damping}"/>
+    </joint>
+    <link name="${name}_link_3_l">
       <inertial>
         <origin xyz="0 0 0" rpy="0 0 0"/>
@@ -392,5 +341,4 @@
       </collision>
     </link>
-   <!-- joint between link_3_l and link_4_l -->
     <joint name="${name}_joint_3_l" type="revolute">
       <parent link="${name}_link_3_l"/>
@@ -398,13 +346,8 @@
       <origin xyz="-0.04188 0.0 0.07873" rpy="${PI / 2} -${PI / 2} 0.0"/>
       <axis xyz="0 0 1"/>
-      <limit lower="${-123.5 * PI / 180}" upper="${80 * PI / 180}"
-             effort="${max_effort}" velocity="${180 * PI / 180}" />
-      <!--   <safety_controller soft_lower_limit="${-168 * M_PI / 180}"
-           soft_upper_limit="${168 * M_PI / 180}"
-           k_position="${safety_controller_k_pos}"
-           k_velocity="${safety_controller_k_vel}"/> -->
-      <dynamics damping="${joint_damping}"/>
-    </joint>
-   <link name="${name}_link_4_l">
+      <limit lower="${-123.5 * PI / 180}" upper="${80 * PI / 180}" effort="${max_effort}" velocity="${180 * PI / 180}" />
+      <dynamics damping="${joint_damping}"/>
+    </joint>
+    <link name="${name}_link_4_l">
       <inertial>
         <origin xyz="0 0 0" rpy="0 0 0"/>
@@ -427,5 +370,4 @@
       </collision>
     </link>
-   <!-- joint between link_4_l and link_5_l -->
     <joint name="${name}_joint_4_l" type="revolute">
       <parent link="${name}_link_4_l"/>
@@ -433,13 +375,8 @@
       <origin xyz="0.0405 0.16461 0.0" rpy="-${PI / 2} 0.0 0.0"/>
       <axis xyz="0 0 1"/>
-      <limit lower="${-290 * PI / 180}" upper="${290 * PI / 180}"
-             effort="${max_effort}" velocity="${400 * PI / 180}" />
-      <!--   <safety_controller soft_lower_limit="${-168 * M_PI / 180}"
-           soft_upper_limit="${168 * M_PI / 180}"
-           k_position="${safety_controller_k_pos}"
-           k_velocity="${safety_controller_k_vel}"/> -->
-      <dynamics damping="${joint_damping}"/>
-    </joint>
-   <link name="${name}_link_5_l">
+      <limit lower="${-290 * PI / 180}" upper="${290 * PI / 180}" effort="${max_effort}" velocity="${400 * PI / 180}" />
+      <dynamics damping="${joint_damping}"/>
+    </joint>
+    <link name="${name}_link_5_l">
       <inertial>
         <origin xyz="0 0 0" rpy="0 0 0"/>
@@ -462,5 +399,4 @@
       </collision>
     </link>
-   <!-- joint between link_5_l and link_6_l -->
     <joint name="${name}_joint_5_l" type="revolute">
       <parent link="${name}_link_5_l"/>
@@ -468,13 +404,8 @@
       <origin xyz="-0.027 0 0.10039" rpy="${PI / 2} 0.0 0.0"/>
       <axis xyz="0 0 1"/>
-      <limit lower="${-88 * PI / 180}" upper="${138 * PI / 180}"
-             effort="${max_effort}" velocity="${400 * PI / 180}" />
-      <!--   <safety_controller soft_lower_limit="${-168 * M_PI / 180}"
-           soft_upper_limit="${168 * M_PI / 180}"
-           k_position="${safety_controller_k_pos}"
-           k_velocity="${safety_controller_k_vel}"/> -->
-      <dynamics damping="${joint_damping}"/>
-    </joint>
-   <link name="${name}_link_6_l">
+      <limit lower="${-88 * PI / 180}" upper="${138 * PI / 180}" effort="${max_effort}" velocity="${400 * PI / 180}" />
+      <dynamics damping="${joint_damping}"/>
+    </joint>
+    <link name="${name}_link_6_l">
       <inertial>
         <origin xyz="0 0 0" rpy="0 0 0"/>
@@ -497,5 +428,4 @@
       </collision>
     </link>
-   <!-- joint between link_6_l and link_7_l -->
     <joint name="${name}_joint_6_l" type="revolute">
       <parent link="${name}_link_6_l"/>
@@ -503,13 +433,8 @@
       <origin xyz="0.027 0.029 0.0" rpy="${-PI / 2} 0.0 0.0"/>
       <axis xyz="0 0 1"/>
-      <limit lower="${-229 * PI / 180}" upper="${229 * PI / 180}"
-             effort="${max_effort}" velocity="${400 * PI / 180}" />
-      <!--   <safety_controller soft_lower_limit="${-168 * M_PI / 180}"
-           soft_upper_limit="${168 * M_PI / 180}"
-           k_position="${safety_controller_k_pos}"
-           k_velocity="${safety_controller_k_vel}"/> -->
-      <dynamics damping="${joint_damping}"/>
-    </joint>
-   <link name="${name}_link_7_l">
+      <limit lower="${-229 * PI / 180}" upper="${229 * PI / 180}" effort="${max_effort}" velocity="${400 * PI / 180}" />
+      <dynamics damping="${joint_damping}"/>
+    </joint>
+    <link name="${name}_link_7_l">
       <inertial>
         <origin xyz="0 0 0" rpy="0 0 0"/>
@@ -532,6 +457,7 @@
       </collision>
     </link>
-    <!--Extensions -->
-    <xacro:yumi_gazebo name="${name}" />
+    <!--                            -->
+    <!--   YuMi Body Transmission   -->
+    <!--                            -->
     <xacro:yumi_transmission name="${name}" hardware_interface="${hardware_interface}"/>
   </xacro:macro>

File: yumi_description/urdf/yumi_servo_gripper.transmission.xacro (robot description, xacro)
@@ -2,12 +2,12 @@
 <robot name="yumi_servo_gripper" xmlns:xacro="http://www.ros.org/wiki/xacro">
   <xacro:macro name="yumi_servo_gripper_transmission" params="name hardware_interface">
-   <transmission name="${name}_tran_1">
+    <transmission name="${name}_tran_1">
       <type>transmission_interface/SimpleTransmission</type>
       <joint name="${name}_joint_1">
-	<hardwareInterface>${hardware_interface}</hardwareInterface>
+        <hardwareInterface>${hardware_interface}</hardwareInterface>
       </joint>
       <actuator name="${name}_motor_1">
-	<hardwareInterface>${hardware_interface}</hardwareInterface>
-	<mechanicalReduction>1</mechanicalReduction>
+        <hardwareInterface>${hardware_interface}</hardwareInterface>
+        <mechanicalReduction>1</mechanicalReduction>
       </actuator>
     </transmission>

File: yumi_description/urdf/yumi_servo_gripper.xacro (robot description, xacro)
@@ -1,17 +1,22 @@
 <?xml version="1.0"?>
+<!--
+  PROGRAMMER: Frederick Wachter
+  DATE CREATED: 2016-05-30
+  LAST MODIFIED: 2016-05-30
+  PURPOSE: Provide colors for the different objects in the YuMi workspace
+  REFERENCE: https://github.com/rtkg/yumi
+-->
 <robot name="yumi" xmlns:xacro="http://www.ros.org/wiki/xacro">
-  <!-- Import all Gazebo-customization elements, including Gazebo colors -->
-  <xacro:include filename="$(find yumi_description)/urdf/yumi_servo_gripper.gazebo.xacro" />
   <!-- Import Transmissions -->
-  <xacro:include filename="$(find yumi_description)/urdf/yumi_servo_gripper.transmission.xacro" />
+  <xacro:include filename="$(find yumi_description)/urdf/yumi_servo_gripper.transmission.xacro"/>
   <!-- Include Utilities -->
   <xacro:include filename="$(find yumi_description)/urdf/utilities.xacro" />
-  <!-- some constants -->
- <!-- <xacro:property name="safety_controller_k_pos" value="100" />
-  <xacro:property name="safety_controller_k_vel" value="2" /> -->
+  <!-- Constants -->
   <xacro:property name="joint_damping" value="0.5" />
   <xacro:property name="max_effort" value="300"/>
   <xacro:macro name="yumi_servo_gripper" params="parent name hardware_interface *origin">
-    <!--joint between {parent} and base-->
+    <!--                         -->
+    <!--      YuMi Gripper       -->
+    <!--                         -->
     <joint name="${parent}_joint" type="fixed">
       <insert_block name="origin"/>
@@ -40,5 +45,4 @@
       </collision>
     </link>
-    <!-- joint between base and right finger -->
     <joint name="${name}_joint" type="prismatic">
       <parent link="${name}_base"/>
@@ -46,10 +50,5 @@
       <origin xyz="0 -0.0065 0.0837" rpy="0 0 0"/>
       <axis xyz="-1 0 0"/>
-      <limit lower="0" upper="0.025"
-             effort="${max_effort}" velocity="0.02" />
-      <!--   <safety_controller soft_lower_limit="${-168 * M_PI / 180}"
-           soft_upper_limit="${168 * M_PI / 180}"
-           k_position="${safety_controller_k_pos}"
-           k_velocity="${safety_controller_k_vel}"/> -->
+      <limit lower="0" upper="0.025" effort="${max_effort}" velocity="0.02" />
       <dynamics damping="${joint_damping}"/>
     </joint>
@@ -75,5 +74,4 @@
       </collision>
     </link>
-   <!-- joint between base and left finger -->
     <joint name="${name}_joint_m" type="prismatic">
       <parent link="${name}_base"/>
@@ -81,10 +79,5 @@
       <origin xyz="0 0.0065 0.0837" rpy="0 0 ${PI}"/>
       <axis xyz="-1 0 0"/>
-      <limit lower="0" upper="0.025"
-             effort="${max_effort}" velocity="0.02" />
-      <!--   <safety_controller soft_lower_limit="${-168 * M_PI / 180}"
-           soft_upper_limit="${168 * M_PI / 180}"
-           k_position="${safety_controller_k_pos}"
-           k_velocity="${safety_controller_k_vel}"/> -->
+      <limit lower="0" upper="0.025" effort="${max_effort}" velocity="0.02" />
       <dynamics damping="${joint_damping}"/>
       <mimic joint="${name}_joint"/>
@@ -111,38 +104,7 @@
       </collision>
     </link>
-    <!-- joint between palm and left finger -->
-    <!--joint name="${name}_joint_2" type="revolute">
-      <parent link="${name}_palm"/>
-      <child link="${name}_left"/>
-      <origin xyz="0.121 0.016 0.0" rpy="${PI} 0 ${PI / 2}"/>
-      <axis xyz="0 0 1"/>
-      <limit lower="${0 * PI / 180}" upper="${90 * PI / 180}"
-             effort="${max_effort}" velocity="${max_velocity}" />
-      <dynamics damping="${joint_damping}"/>
-      <mimic joint="${name}_joint_1"/>
-    </joint>
-    <link name="${name}_left">
-      <inertial>
-        <origin xyz="0.01 0 0" rpy="0 0 0"/>
-        <mass value="0.5"/>
-        <inertia ixx="0.001"  ixy="0"  ixz="0" iyy="0.001" iyz="0" izz="0.001" />
-      </inertial>
-      <visual>
-        <origin xyz="0 0 0" rpy="0 0 0"/>
-        <geometry>
-          <mesh filename="package://velvet_fingers_description/meshes/velvet_fingers_left.stl"/>
-        </geometry>
-        <material name="VELVET_FINGERS/Orange"/>
-      </visual>
-      <collision>
-        <origin xyz="0 0 0" rpy="0 0 0"/>
-        <geometry>
-          <mesh filename="package://velvet_fingers_description/meshes/velvet_fingers_left.stl"/>
-        </geometry>
-        <material name="VELVET_FINGERS/Orange"/>
-      </collision>
-    </link-->
-     <!--Extensions -->
-    <xacro:yumi_servo_gripper_gazebo name="${name}" />
+    <!--                               -->
+    <!--   YuMi Gripper Transmission   -->
+    <!--                               -->
     <xacro:yumi_servo_gripper_transmission name="${name}" hardware_interface="${hardware_interface}"/>
   </xacro:macro>
