Commit message: modified launch files

File: yumi_description/urdf/yumi_servo_gripper.xacro (robot description, xacro)
@@ -111,36 +111,4 @@
       </collision>
     </link>
-    <!-- joint between palm and left finger -->
-    <!--joint name="${name}_joint_2" type="revolute">
-      <parent link="${name}_palm"/>
-      <child link="${name}_left"/>
-      <origin xyz="0.121 0.016 0.0" rpy="${PI} 0 ${PI / 2}"/>
-      <axis xyz="0 0 1"/>
-      <limit lower="${0 * PI / 180}" upper="${90 * PI / 180}"
-             effort="${max_effort}" velocity="${max_velocity}" />
-      <dynamics damping="${joint_damping}"/>
-      <mimic joint="${name}_joint_1"/>
-    </joint>
-    <link name="${name}_left">
-      <inertial>
-        <origin xyz="0.01 0 0" rpy="0 0 0"/>
-        <mass value="0.5"/>
-        <inertia ixx="0.001"  ixy="0"  ixz="0" iyy="0.001" iyz="0" izz="0.001" />
-      </inertial>
-      <visual>
-        <origin xyz="0 0 0" rpy="0 0 0"/>
-        <geometry>
-          <mesh filename="package://velvet_fingers_description/meshes/velvet_fingers_left.stl"/>
-        </geometry>
-        <material name="VELVET_FINGERS/Orange"/>
-      </visual>
-      <collision>
-        <origin xyz="0 0 0" rpy="0 0 0"/>
-        <geometry>
-          <mesh filename="package://velvet_fingers_description/meshes/velvet_fingers_left.stl"/>
-        </geometry>
-        <material name="VELVET_FINGERS/Orange"/>
-      </collision>
-    </link-->
      <!--Extensions -->
     <xacro:yumi_servo_gripper_gazebo name="${name}" />

Commit message: friction tweaks

File: yumi_description/urdf/yumi_servo_gripper.xacro (robot description, xacro)
@@ -10,6 +10,7 @@
  <!-- <xacro:property name="safety_controller_k_pos" value="100" />
   <xacro:property name="safety_controller_k_vel" value="2" /> -->
-  <xacro:property name="joint_damping" value="0.5" />
-  <xacro:property name="max_effort" value="300"/>
+  <xacro:property name="gripper_joint_damping" value="1.0" />
+  <xacro:property name="max_gripper_effort" value="50"/>
+<xacro:property name="max_gripper_velocity" value="2"/>
   <xacro:macro name="yumi_servo_gripper" params="parent name hardware_interface *origin">
     <!--joint between {parent} and base-->
@@ -47,10 +48,10 @@
       <axis xyz="-1 0 0"/>
       <limit lower="0" upper="0.025"
-             effort="${max_effort}" velocity="0.02" />
+             effort="${max_gripper_effort}" velocity="${max_gripper_velocity}" />
       <!--   <safety_controller soft_lower_limit="${-168 * M_PI / 180}"
            soft_upper_limit="${168 * M_PI / 180}"
            k_position="${safety_controller_k_pos}"
            k_velocity="${safety_controller_k_vel}"/> -->
-      <dynamics damping="${joint_damping}"/>
+      <dynamics damping="${gripper_joint_damping}"/>
     </joint>
     <link name="${name}_finger_r">
@@ -75,4 +76,15 @@
       </collision>
     </link>
+  <gazebo reference="${name}_finger_r">
+    <material>Gazebo/Blue</material>
+    <turnGravityOff>false</turnGravityOff>
+    <kp>1000000.0</kp>
+    <kd>1.0</kd>
+    <mu1>30000.0</mu1>
+    <mu2>30000.0</mu2>
+    <selfCollide>false</selfCollide>
+    <maxContacts>10</maxContacts>
+    <minDepth>0.001</minDepth>
+  </gazebo>
    <!-- joint between base and left finger -->
     <joint name="${name}_joint_m" type="prismatic">
@@ -82,10 +94,10 @@
       <axis xyz="-1 0 0"/>
       <limit lower="0" upper="0.025"
-             effort="${max_effort}" velocity="0.02" />
+             effort="${max_gripper_effort}" velocity="${max_gripper_velocity}" />
       <!--   <safety_controller soft_lower_limit="${-168 * M_PI / 180}"
            soft_upper_limit="${168 * M_PI / 180}"
            k_position="${safety_controller_k_pos}"
            k_velocity="${safety_controller_k_vel}"/> -->
-      <dynamics damping="${joint_damping}"/>
+      <dynamics damping="${gripper_joint_damping}"/>
       <mimic joint="${name}_joint"/>
     </joint>
@@ -111,4 +123,15 @@
       </collision>
     </link>
+  <gazebo reference="${name}_finger_l">
+    <material>Gazebo/Blue</material>
+    <turnGravityOff>false</turnGravityOff>
+    <kp>1000000.0</kp>
+    <kd>1.0</kd>
+    <mu1>30000.0</mu1>
+    <mu2>30000.0</mu2>
+    <selfCollide>false</selfCollide>
+    <maxContacts>10</maxContacts>
+    <minDepth>0.001</minDepth>
+  </gazebo>
      <!--Extensions -->
     <xacro:yumi_servo_gripper_gazebo name="${name}" />
