Commit message: Added a new link without inertia as the yumi base, so that MoveIt! works properly. Updated MoveIt! config files.

File: yumi_description/urdf/yumi.urdf (robot description, URDF)
Before this commit: robot yumi, 22 links, 21 joints
Links:
- removed link world
- added link yumi_base_link
Joints:
- removed joint world_joint
- added joint yumi_base_link_to_body: type fixed, parent yumi_base_link, child yumi_body, origin xyz=0 0 0 rpy=0 0 0
- joint gripper_l_joint: limit lower=0 upper=0.025 effort=50 velocity=2 -> lower=0 upper=0.025 effort=20 velocity=2
- joint gripper_l_joint_m: limit lower=0 upper=0.025 effort=50 velocity=2 -> lower=0 upper=0.025 effort=20 velocity=2
- joint gripper_r_joint: limit lower=0 upper=0.025 effort=50 velocity=2 -> lower=0 upper=0.025 effort=20 velocity=2
- joint gripper_r_joint_m: limit lower=0 upper=0.025 effort=50 velocity=2 -> lower=0 upper=0.025 effort=20 velocity=2

File: yumi_description/urdf/yumi.urdf.xacro (robot description, xacro)
@@ -28,7 +28,7 @@
     <link name="world"/>
     <joint name="world_joint" type="fixed">
+      <parent link="world"/>
+      <child link="yumi_base_link"/>
       <origin xyz="0 0 0.1" rpy="0 0 0" />
-      <parent link="world"/>
-      <child link="yumi_body"/>
     </joint>
   </xacro:if>
@@ -42,7 +42,7 @@
     <link name="world"/>
     <joint name="world_to_pedestal" type="fixed">
-      <origin rpy="0 0 0" xyz="0 0 ${pedestal_height}" />
       <parent link="world" />
       <child link="yumi_pedestal" />
+      <origin rpy="0 0 0" xyz="0 0 ${pedestal_height}" />
     </joint>
     <link name="yumi_pedestal">
@@ -63,7 +63,7 @@
     </link>
     <joint name="pedestal_to_yumi" type="fixed">
+      <parent link="yumi_pedestal" />
+      <child link="yumi_base_link" />
       <origin rpy="0 0 0" xyz="${yumi_offset_x} 0 ${yumi_height}" />
-      <parent link="yumi_pedestal" />
-      <child link="yumi_body" />
     </joint>
   </xacro:if>
@@ -78,7 +78,7 @@
     <link name="world"/>
     <joint name="world_to_pedestal" type="fixed">
-      <origin rpy="0 0 0" xyz="0 0 ${pedestal_height}" />
       <parent link="world" />
       <child link="yumi_pedestal" />
+      <origin rpy="0 0 0" xyz="0 0 ${pedestal_height}" />
     </joint>
     <link name="yumi_pedestal">
@@ -92,7 +92,7 @@
     </link>
     <joint name="pedestal_to_table" type="fixed">
-      <origin rpy="0 0 0" xyz="0.235 0 ${yumi_height}" />
       <parent link="yumi_pedestal" />
       <child link="table" />
+      <origin rpy="0 0 0" xyz="0.235 0 ${yumi_height}" />
     </joint>
     <link name="table">
@@ -106,7 +106,7 @@
     </link>
     <joint name="pedestal_to_yumi" type="fixed">
+      <parent link="yumi_pedestal" />
+      <child link="yumi_base_link" />
       <origin rpy="0 0 0" xyz="${yumi_offset_x} 0 ${yumi_height+0.02}" />
-      <parent link="yumi_pedestal" />
-      <child link="yumi_body" />
     </joint>
     <link name="kinect2">
@@ -147,22 +147,22 @@
     </link>
      <joint name="kinect2_to_right_kinect_base" type="fixed">
+      <parent link="yumi_base_link" />
+      <child link="right_kinect_base" />
       <origin rpy="0 ${-PI/6} 0.17" xyz="0.1 -0.03 0.56" />
-      <parent link="yumi_body" />
-      <child link="right_kinect_base" />
     </joint>
     <joint name="kinect2_to_left_kinect_base" type="fixed">
+      <parent link="yumi_base_link" />
+      <child link="left_kinect_base" />
       <origin rpy="0 ${-PI/6} -0.17" xyz="0.1 0.03 0.56" />
-      <parent link="yumi_body" />
-      <child link="left_kinect_base" />
     </joint>
     <joint name="yumi_to_middle_kinect_base" type="fixed">
+      <parent link="yumi_base_link" />
+      <child link="middle_kinect_base" />
       <origin rpy="0 ${-PI/6} 0" xyz="0.05 0 0.56" />
-      <parent link="yumi_body" />
-      <child link="middle_kinect_base" />
     </joint>
     <joint name="middle_kinect_base_to_kinect2" type="fixed">
-      <origin rpy="${-PI/2} 0 ${kinect_zrotation_fix}" xyz="0.2 0 0" />
       <parent link="middle_kinect_base" />
       <child link="kinect2" />
+      <origin rpy="${-PI/2} 0 ${kinect_zrotation_fix}" xyz="0.2 0 0" />
     </joint>
   </xacro:if>

File: yumi_description/urdf/yumi.xacro (robot description, xacro)
@@ -9,4 +9,10 @@
   <xacro:property name="max_effort" value="300"/>
   <xacro:macro name="yumi" params="parent name hardware_interface *origin">
+    <link name="yumi_base_link"></link>
+    <joint name="${name}_base_link_to_body" type="fixed">
+      <parent link="yumi_base_link"/>
+      <child link="${name}_body"/>
+      <origin xyz="0 0 0" rpy="0 0 0"/>
+    </joint>
     <link name="${name}_body">
       <inertial>

Commit message: Added YuMi end effectors to MoveIt! config

File: yumi_description/urdf/yumi.urdf (robot description, URDF)
Before this commit: robot yumi, 22 links, 21 joints
Links:
- added link world
Joints:
- added joint world_joint: type fixed, parent world, child yumi_base_link, origin xyz=0 0 0.1 rpy=0 0 0
