Commit message: Cleaned up in the code

File: yumi_description/urdf/yumi.gazebo.xacro (robot description, xacro)
@@ -8,4 +8,117 @@
       <mu2>0.2</mu2>
     </gazebo>
+  <gazebo reference= "${name}_link_1_r">
+    <sensor name="${name}_link_1_r_bumper" type="contact">
+      <always_on>true</always_on>
+      <update_rate>100</update_rate>
+      <contact>
+        <collision>${name}_link_1_r_collision</collision>
+      </contact>
+      <plugin filename="libgazebo_ros_bumper.so" name="${name}_link_1_r_plugin">
+        <always_on>1</always_on>
+        <update_rate>100</update_rate>
+        <frameName>${name}_link_1_r</frameName>
+        <bumperTopicName>${name}/link_1_r/contact</bumperTopicName>
+      </plugin>
+    </sensor>
+    <material>Gazebo/Orange</material>
+  </gazebo>
+    <gazebo reference= "${name}_link_2_r">
+    <sensor name="${name}_link_2_r_bumper" type="contact">
+      <always_on>true</always_on>
+      <update_rate>100</update_rate>
+      <contact>
+        <collision>${name}_link_2_r_collision</collision>
+      </contact>
+      <plugin filename="libgazebo_ros_bumper.so" name="${name}_link_2_r_plugin">
+        <always_on>1</always_on>
+        <update_rate>100</update_rate>
+        <frameName>${name}_link_2_r</frameName>
+        <bumperTopicName>${name}/link_2_r/contact</bumperTopicName>
+      </plugin>
+    </sensor>
+    <material>Gazebo/Orange</material>
+  </gazebo>
+    <gazebo reference= "${name}_link_3_r">
+    <sensor name="${name}_link_3_r_bumper" type="contact">
+      <always_on>true</always_on>
+      <update_rate>100</update_rate>
+      <contact>
+        <collision>${name}_link_3_r_collision</collision>
+      </contact>
+      <plugin filename="libgazebo_ros_bumper.so" name="${name}_link_3_r_plugin">
+        <always_on>1</always_on>
+        <update_rate>100</update_rate>
+        <frameName>${name}_link_3_r</frameName>
+        <bumperTopicName>${name}/link_3_r/contact</bumperTopicName>
+      </plugin>
+    </sensor>
+    <material>Gazebo/Orange</material>
+  </gazebo>
+    <gazebo reference= "${name}_link_4_r">
+    <sensor name="${name}_link_4_r_bumper" type="contact">
+      <always_on>true</always_on>
+      <update_rate>100</update_rate>
+      <contact>
+        <collision>${name}_link_4_r_collision</collision>
+      </contact>
+      <plugin filename="libgazebo_ros_bumper.so" name="${name}_link_4_r_plugin">
+        <always_on>1</always_on>
+        <update_rate>100</update_rate>
+        <frameName>${name}_link_4_r</frameName>
+        <bumperTopicName>${name}/link_4_r/contact</bumperTopicName>
+      </plugin>
+    </sensor>
+    <material>Gazebo/Orange</material>
+  </gazebo>
+    <gazebo reference= "${name}_link_5_r">
+    <sensor name="${name}_link_5_r_bumper" type="contact">
+      <always_on>true</always_on>
+      <update_rate>100</update_rate>
+      <contact>
+        <collision>${name}_link_5_r_collision</collision>
+      </contact>
+      <plugin filename="libgazebo_ros_bumper.so" name="${name}_link_5_r_plugin">
+        <always_on>1</always_on>
+        <update_rate>100</update_rate>
+        <frameName>${name}_link_5_r</frameName>
+        <bumperTopicName>${name}/link_5_r/contact</bumperTopicName>
+      </plugin>
+    </sensor>
+    <material>Gazebo/Orange</material>
+  </gazebo>
+    <gazebo reference= "${name}_link_6_r">
+    <sensor name="${name}_link_6_r_bumper" type="contact">
+      <always_on>true</always_on>
+      <update_rate>100</update_rate>
+      <contact>
+        <collision>${name}_link_6_r_collision</collision>
+      </contact>
+      <plugin filename="libgazebo_ros_bumper.so" name="${name}_link_6_r_plugin">
+        <always_on>1</always_on>
+        <update_rate>100</update_rate>
+        <frameName>${name}_link_6_r</frameName>
+        <bumperTopicName>${name}/link_6_r/contact</bumperTopicName>
+      </plugin>
+    </sensor>
+    <material>Gazebo/Orange</material>
+  </gazebo>
+    <gazebo reference= "${name}_link_7_r">
+    <sensor name="${name}_link_7_r_bumper" type="contact">
+      <always_on>true</always_on>
+      <update_rate>100</update_rate>
+      <contact>
+        <collision>yumi_link_7_l_collision</collision>
+        <topic>/bumper_contact</topic>
+      </contact>
+      <plugin filename="libgazebo_ros_bumper.so" name="${name}_link_7_r_plugin">
+        <always_on>1</always_on>
+        <update_rate>100</update_rate>
+        <frameName>${name}_link_7_r</frameName>
+        <bumperTopicName>${name}/link_7_r/contact</bumperTopicName>
+      </plugin>
+    </sensor>
+    <material>Gazebo/Orange</material>
+  </gazebo>
   </xacro:macro>
 </robot>

File: yumi_description/urdf/yumi.urdf.xacro (robot description, xacro)
@@ -9,26 +9,14 @@
   <!--Import the yumi servo gripper macro -->
   <xacro:include filename="$(find yumi_description)/urdf/yumi_servo_gripper.xacro"/>
-  <!--Import the yumi camera macro -->
-  <!-- <xacro:include filename="$(find yumi_description)/urdf/yumi_camera.xacro"/> -->
-  <!--Import the table macro -->
-  <!-- <xacro:include filename="$(find yumi_description)/urdf/yumi_table.urdf.xacro"/> -->
-  <!--Import the box macro -->
-  <!-- <xacro:include filename="$(find yumi_description)/urdf/object.urdf.xacro"/> -->
-  <!-- Import Gazebo plugins -->
+ <!-- Import Gazebo plugins -->
   <xacro:include filename="$(find yumi_description)/gazebo/gazebo.urdf.xacro"/>
+ <!-- Import table  -->
+  <xacro:include filename="$(find yumi_description)/urdf/yumi_table.urdf.xacro"/>
   <!-- Fix to world just for testing -->
   <link name="world"/>
-  <!--Define the table height-->
-  <property name="table_height_from_gound" value="0.89" />
-  <!--table-->
-  <!-- <xacro:yumi_table parent="world" table_height="${table_height_from_gound}"/> -->
-  <!--box-->
-<!--   <xacro:yumi_box parent="table_top_link">
-    <origin xyz="0.5 0 ${table_height_from_gound+0.1}" rpy="0 0 0" />
-  </xacro:yumi_box>
- -->
+  <xacro:yumi_table parent="world" table_height="0.6"/>
   <!--yumi-->
   <xacro:yumi name="yumi" hardware_interface="$(arg prefix)" parent="world">
-    <origin xyz="0 0 ${table_height_from_gound}" rpy="0 0 0" />
+    <origin xyz="0 0 0.1" rpy="0 0 0" />
   </xacro:yumi>
   <!--right gripper-->
@@ -40,7 +28,3 @@
     <origin xyz="0 0 0.007" rpy="0 0 ${PI}" />
   </xacro:yumi_servo_gripper>
-<!--   <xacro:yumi_camera name="yumi_top_camera" parent="world">
-    <origin xyz="0.883 -0.06 ${0.877+table_height_from_gound}" rpy="3.12 0.795 0.005" />
-  </xacro:yumi_camera>
- -->
 </robot>

File: yumi_description/urdf/yumi.xacro (robot description, xacro)
@@ -276,5 +276,5 @@
           <mesh filename="package://yumi_description/meshes/link_7.stl"/>
         </geometry>
-        <material name="Grey"/>
+        <material name="Blue"/>
       </visual>
       <collision>
