Commit message: one arm done

File: yumi_description/urdf/yumi.xacro (robot description, xacro)
@@ -180,4 +180,109 @@
       </collision>
     </link>
+   <!-- joint between link_4_r and link_5_r -->
+    <joint name="${name}_joint_5_r" type="revolute">
+      <parent link="${name}_link_4_r"/>
+      <child link="${name}_link_5_r"/>
+      <origin xyz="0.0405 0.16461 0.0" rpy="-1.5708 0.0 0.0"/>
+      <axis xyz="0 0 1"/>
+      <limit lower="${-290 * PI / 180}" upper="${290 * PI / 180}"
+             effort="${max_effort}" velocity="${400 * PI / 180}" />
+      <!--   <safety_controller soft_lower_limit="${-168 * M_PI / 180}"
+           soft_upper_limit="${168 * M_PI / 180}"
+           k_position="${safety_controller_k_pos}"
+           k_velocity="${safety_controller_k_vel}"/> -->
+      <dynamics damping="${joint_damping}"/>
+    </joint>
+   <link name="${name}_link_5_r">
+      <inertial>
+        <origin xyz="0 0 0" rpy="0 0 0"/>
+        <mass value="2"/>
+        <inertia ixx="0.1"  ixy="0"  ixz="0" iyy="0.1" iyz="0" izz="0.1" />
+      </inertial>
+      <visual>
+        <origin xyz="0 0 0" rpy="0 0 0"/>
+        <geometry>
+          <mesh filename="package://yumi_description/meshes/link_5.stl"/>
+        </geometry>
+        <material name="Grey"/>
+      </visual>
+      <collision>
+        <origin xyz="0 0 0" rpy="0 0 0"/>
+        <geometry>
+          <mesh filename="package://yumi_description/meshes/coarse/link_5.stl"/>
+        </geometry>
+        <material name="Grey"/>
+      </collision>
+    </link>
+   <!-- joint between link_5_r and link_6_r -->
+    <joint name="${name}_joint_6_r" type="revolute">
+      <parent link="${name}_link_5_r"/>
+      <child link="${name}_link_6_r"/>
+      <origin xyz="-0.027 0 0.10039" rpy="1.5708 0.0 0.0"/>
+      <axis xyz="0 0 1"/>
+      <limit lower="${-88 * PI / 180}" upper="${138 * PI / 180}"
+             effort="${max_effort}" velocity="${400 * PI / 180}" />
+      <!--   <safety_controller soft_lower_limit="${-168 * M_PI / 180}"
+           soft_upper_limit="${168 * M_PI / 180}"
+           k_position="${safety_controller_k_pos}"
+           k_velocity="${safety_controller_k_vel}"/> -->
+      <dynamics damping="${joint_damping}"/>
+    </joint>
+   <link name="${name}_link_6_r">
+      <inertial>
+        <origin xyz="0 0 0" rpy="0 0 0"/>
+        <mass value="2"/>
+        <inertia ixx="0.1"  ixy="0"  ixz="0" iyy="0.1" iyz="0" izz="0.1" />
+      </inertial>
+      <visual>
+        <origin xyz="0 0 0" rpy="0 0 0"/>
+        <geometry>
+          <mesh filename="package://yumi_description/meshes/link_6.stl"/>
+        </geometry>
+        <material name="Grey"/>
+      </visual>
+      <collision>
+        <origin xyz="0 0 0" rpy="0 0 0"/>
+        <geometry>
+          <mesh filename="package://yumi_description/meshes/coarse/link_6.stl"/>
+        </geometry>
+        <material name="Grey"/>
+      </collision>
+    </link>
+   <!-- joint between link_6_r and link_7_r -->
+    <joint name="${name}_joint_7_r" type="revolute">
+      <parent link="${name}_link_6_r"/>
+      <child link="${name}_link_7_r"/>
+      <origin xyz="0.027 0.029 0.0" rpy="-1.5708 0.0 0.0"/>
+      <axis xyz="0 0 1"/>
+      <limit lower="${-229 * PI / 180}" upper="${229 * PI / 180}"
+             effort="${max_effort}" velocity="${400 * PI / 180}" />
+      <!--   <safety_controller soft_lower_limit="${-168 * M_PI / 180}"
+           soft_upper_limit="${168 * M_PI / 180}"
+           k_position="${safety_controller_k_pos}"
+           k_velocity="${safety_controller_k_vel}"/> -->
+      <dynamics damping="${joint_damping}"/>
+    </joint>
+   <link name="${name}_link_7_r">
+      <inertial>
+        <origin xyz="0 0 0" rpy="0 0 0"/>
+        <mass value="2"/>
+        <inertia ixx="0.1"  ixy="0"  ixz="0" iyy="0.1" iyz="0" izz="0.1" />
+      </inertial>
+      <visual>
+        <origin xyz="0 0 0" rpy="0 0 0"/>
+        <geometry>
+          <mesh filename="package://yumi_description/meshes/link_7.stl"/>
+        </geometry>
+        <material name="Grey"/>
+      </visual>
+      <collision>
+        <origin xyz="0 0 0" rpy="0 0 0"/>
+        <geometry>
+          <mesh filename="package://yumi_description/meshes/coarse/link_7.stl"/>
+        </geometry>
+        <material name="Grey"/>
+      </collision>
+    </link>
     <!--Extensions -->
     <xacro:yumi_gazebo name="${name}" />

Commit message: Add a tool frame to both hands.

File: yumi_description/urdf/yumi.xacro (robot description, xacro)
@@ -285,5 +285,12 @@
         <material name="Grey"/>
       </collision>
-    </link>
+   </link>
+   <!-- A Tool frame -->
+   <joint name="${name}_joint_tool_r" type="fixed">
+     <parent link="${name}_link_7_r"/>
+     <child link="${name}_link_tool_r"/>
+     <origin xyz="0.0 0.0 0.1" rpy="-${PI / 2} -${PI / 2} 0.0"/>
+   </joint>
+   <link name="${name}_link_tool_r"/>
    <!--///////////////////////////////////// LEFT ARM ////////////////////////////////  -->
   <!-- joint between body and link_1_l -->
@@ -531,5 +538,11 @@
         <material name="Grey"/>
       </collision>
-    </link>
+   </link>
+   <joint name="${name}_joint_tool_l" type="fixed">
+     <parent link="${name}_link_7_l"/>
+     <child link="${name}_link_tool_l"/>
+     <origin xyz="0.0 0.0 0.1" rpy="-${PI / 2} -${PI / 2} 0.0"/>
+   </joint>
+   <link name="${name}_link_tool_l"/>
     <!--Extensions -->
     <xacro:yumi_gazebo name="${name}" />

Commit message: Changes to make ridgeback_yumi pkg work

File: yumi_description/urdf/yumi.xacro (robot description, xacro)
@@ -6,15 +6,15 @@
   <xacro:include filename="$(find yumi_description)/urdf/yumi.transmission.xacro" />
   <!-- some constants -->
- <!-- <xacro:property name="safety_controller_k_pos" value="100" />
-  <xacro:property name="safety_controller_k_vel" value="2" /> -->
   <xacro:property name="joint_damping" value="0.5" />
   <xacro:property name="max_effort" value="300"/>
   <xacro:macro name="yumi" params="name parent hardware_interface *origin">
-    <!--joint between {parent} and body-->
-    <joint name="${parent}_joint" type="fixed">
-      <insert_block name="origin"/>
-      <parent link="${parent}"/>
-      <child link="${name}_body"/>
-    </joint>
+    <xacro:if value="${parent == 'world'}">
+      <!--joint between world and body-->
+      <joint name="world_joint" type="fixed">
+        <insert_block name="origin"/>
+        <parent link="world"/>
+        <child link="${name}_body"/>
+      </joint>
+    </xacro:if>
     <link name="${name}_body">
       <inertial>
@@ -88,5 +88,5 @@
       <dynamics damping="${joint_damping}"/>
     </joint>
-   <link name="${name}_link_2_r">
+    <link name="${name}_link_2_r">
       <inertial>
         <origin xyz="0 0 0" rpy="0 0 0"/>
@@ -109,19 +109,15 @@
       </collision>
     </link>
-   <!-- joint between link_2_r and link_3_r -->
-    <joint name="${name}_joint_7_r" type="revolute">
-      <parent link="${name}_link_2_r"/>
-      <child link="${name}_link_3_r"/>
-      <origin xyz="-0.03 0.17283 0.0" rpy="${-PI / 2} 0.0 0.0"/>
-      <axis xyz="0 0 1"/>
-      <limit lower="${-168.5 * PI / 180}" upper="${168.5 * PI / 180}"
-             effort="${max_effort}" velocity="${180 * PI / 180}" />
-      <!--   <safety_controller soft_lower_limit="${-168 * M_PI / 180}"
-           soft_upper_limit="${168 * M_PI / 180}"
-           k_position="${safety_controller_k_pos}"
-           k_velocity="${safety_controller_k_vel}"/> -->
-      <dynamics damping="${joint_damping}"/>
-    </joint>
-   <link name="${name}_link_3_r">
+     <!-- joint between link_2_r and link_3_r -->
+      <joint name="${name}_joint_7_r" type="revolute">
+        <parent link="${name}_link_2_r"/>
+        <child link="${name}_link_3_r"/>
+        <origin xyz="-0.03 0.17283 0.0" rpy="${-PI / 2} 0.0 0.0"/>
+        <axis xyz="0 0 1"/>
+        <limit lower="${-168.5 * PI / 180}" upper="${168.5 * PI / 180}"
+               effort="${max_effort}" velocity="${180 * PI / 180}" />
+        <dynamics damping="${joint_damping}"/>
+      </joint>
+    <link name="${name}_link_3_r">
       <inertial>
         <origin xyz="0 0 0" rpy="0 0 0"/>
@@ -144,5 +140,5 @@
       </collision>
     </link>
-   <!-- joint between link_3_r and link_4_r -->
+    <!-- joint between link_3_r and link_4_r -->
     <joint name="${name}_joint_3_r" type="revolute">
       <parent link="${name}_link_3_r"/>
@@ -152,11 +148,7 @@
       <limit lower="${-123.5 * PI / 180}" upper="${80 * PI / 180}"
              effort="${max_effort}" velocity="${180 * PI / 180}" />
-      <!--   <safety_controller soft_lower_limit="${-168 * M_PI / 180}"
-           soft_upper_limit="${168 * M_PI / 180}"
-           k_position="${safety_controller_k_pos}"
-           k_velocity="${safety_controller_k_vel}"/> -->
-      <dynamics damping="${joint_damping}"/>
-    </joint>
-   <link name="${name}_link_4_r">
+      <dynamics damping="${joint_damping}"/>
+    </joint>
+    <link name="${name}_link_4_r">
       <inertial>
         <origin xyz="0 0 0" rpy="0 0 0"/>
@@ -179,5 +171,5 @@
       </collision>
     </link>
-   <!-- joint between link_4_r and link_5_r -->
+    <!-- joint between link_4_r and link_5_r -->
     <joint name="${name}_joint_4_r" type="revolute">
       <parent link="${name}_link_4_r"/>
@@ -187,11 +179,7 @@
       <limit lower="${-290 * PI / 180}" upper="${290 * PI / 180}"
              effort="${max_effort}" velocity="${400 * PI / 180}" />
-      <!--   <safety_controller soft_lower_limit="${-168 * M_PI / 180}"
-           soft_upper_limit="${168 * M_PI / 180}"
-           k_position="${safety_controller_k_pos}"
-           k_velocity="${safety_controller_k_vel}"/> -->
-      <dynamics damping="${joint_damping}"/>
-    </joint>
-   <link name="${name}_link_5_r">
+      <dynamics damping="${joint_damping}"/>
+    </joint>
+    <link name="${name}_link_5_r">
       <inertial>
         <origin xyz="0 0 0" rpy="0 0 0"/>
@@ -214,5 +202,5 @@
       </collision>
     </link>
-   <!-- joint between link_5_r and link_6_r -->
+    <!-- joint between link_5_r and link_6_r -->
     <joint name="${name}_joint_5_r" type="revolute">
       <parent link="${name}_link_5_r"/>
@@ -222,11 +210,7 @@
       <limit lower="${-88 * PI / 180}" upper="${138 * PI / 180}"
              effort="${max_effort}" velocity="${400 * PI / 180}" />
-      <!--   <safety_controller soft_lower_limit="${-168 * M_PI / 180}"
-           soft_upper_limit="${168 * M_PI / 180}"
-           k_position="${safety_controller_k_pos}"
-           k_velocity="${safety_controller_k_vel}"/> -->
-      <dynamics damping="${joint_damping}"/>
-    </joint>
-   <link name="${name}_link_6_r">
+      <dynamics damping="${joint_damping}"/>
+    </joint>
+    <link name="${name}_link_6_r">
       <inertial>
         <origin xyz="0 0 0" rpy="0 0 0"/>
@@ -249,5 +233,5 @@
       </collision>
     </link>
-   <!-- joint between link_6_r and link_7_r -->
+    <!-- joint between link_6_r and link_7_r -->
     <joint name="${name}_joint_6_r" type="revolute">
       <parent link="${name}_link_6_r"/>
@@ -257,11 +241,7 @@
       <limit lower="${-229 * PI / 180}" upper="${229 * PI / 180}"
              effort="${max_effort}" velocity="${400 * PI / 180}" />
-      <!--   <safety_controller soft_lower_limit="${-168 * M_PI / 180}"
-           soft_upper_limit="${168 * M_PI / 180}"
-           k_position="${safety_controller_k_pos}"
-           k_velocity="${safety_controller_k_vel}"/> -->
-      <dynamics damping="${joint_damping}"/>
-    </joint>
-   <link name="${name}_link_7_r">
+      <dynamics damping="${joint_damping}"/>
+    </joint>
+    <link name="${name}_link_7_r">
       <inertial>
         <origin xyz="0 0 0" rpy="0 0 0"/>
@@ -284,6 +264,6 @@
       </collision>
     </link>
-   <!--///////////////////////////////////// LEFT ARM ////////////////////////////////  -->
-  <!-- joint between body and link_1_l -->
+    <!--///////////////////////////////////// LEFT ARM ////////////////////////////////  -->
+    <!-- joint between body and link_1_l -->
     <joint name="${name}_joint_1_l" type="revolute">
       <parent link="${name}_body"/>
@@ -293,11 +273,7 @@
       <limit lower="${-168.5 * PI / 180}" upper="${168.5 * PI / 180}"
              effort="${max_effort}" velocity="${180 * PI / 180}" />
-      <!--   <safety_controller soft_lower_limit="${-168 * M_PI / 180}"
-           soft_upper_limit="${168 * M_PI / 180}"
-           k_position="${safety_controller_k_pos}"
-           k_velocity="${safety_controller_k_vel}"/> -->
-      <dynamics damping="${joint_damping}"/>
-    </joint>
-   <link name="${name}_link_1_l">
+      <dynamics damping="${joint_damping}"/>
+    </joint>
+    <link name="${name}_link_1_l">
       <inertial>
         <origin xyz="0 -0.03 0.12" rpy="0 0 0"/>
@@ -320,5 +296,5 @@
       </collision>
     </link>
- <!-- joint between link_1_l and link_2_l -->
+    <!-- joint between link_1_l and link_2_l -->
     <joint name="${name}_joint_2_l" type="revolute">
       <parent link="${name}_link_1_l"/>
@@ -328,11 +304,7 @@
       <limit lower="${-143.5 * PI / 180}" upper="${43.5 * PI / 180}"
              effort="${max_effort}" velocity="${180 * PI / 180}" />
-      <!--   <safety_controller soft_lower_limit="${-168 * M_PI / 180}"
-           soft_upper_limit="${168 * M_PI / 180}"
-           k_position="${safety_controller_k_pos}"
-           k_velocity="${safety_controller_k_vel}"/> -->
-      <dynamics damping="${joint_damping}"/>
-    </joint>
-   <link name="${name}_link_2_l">
+      <dynamics damping="${joint_damping}"/>
+    </joint>
+    <link name="${name}_link_2_l">
       <inertial>
         <origin xyz="0 0 0" rpy="0 0 0"/>
@@ -355,5 +327,5 @@
       </collision>
     </link>
- <!-- joint between link_2_l and link_3_l -->
+    <!-- joint between link_2_l and link_3_l -->
     <joint name="${name}_joint_7_l" type="revolute">
       <parent link="${name}_link_2_l"/>
@@ -363,11 +335,7 @@
       <limit lower="${-168.5 * PI / 180}" upper="${168.5 * PI / 180}"
              effort="${max_effort}" velocity="${180 * PI / 180}" />
-      <!--   <safety_controller soft_lower_limit="${-168 * M_PI / 180}"
-           soft_upper_limit="${168 * M_PI / 180}"
-           k_position="${safety_controller_k_pos}"
-           k_velocity="${safety_controller_k_vel}"/> -->
-      <dynamics damping="${joint_damping}"/>
-    </joint>
-   <link name="${name}_link_3_l">
+      <dynamics damping="${joint_damping}"/>
+    </joint>
+    <link name="${name}_link_3_l">
       <inertial>
         <origin xyz="0 0 0" rpy="0 0 0"/>
@@ -390,5 +358,5 @@
       </collision>
     </link>
-   <!-- joint between link_3_l and link_4_l -->
+    <!-- joint between link_3_l and link_4_l -->
     <joint name="${name}_joint_3_l" type="revolute">
       <parent link="${name}_link_3_l"/>
@@ -398,11 +366,7 @@
       <limit lower="${-123.5 * PI / 180}" upper="${80 * PI / 180}"
              effort="${max_effort}" velocity="${180 * PI / 180}" />
-      <!--   <safety_controller soft_lower_limit="${-168 * M_PI / 180}"
-           soft_upper_limit="${168 * M_PI / 180}"
-           k_position="${safety_controller_k_pos}"
-           k_velocity="${safety_controller_k_vel}"/> -->
-      <dynamics damping="${joint_damping}"/>
-    </joint>
-   <link name="${name}_link_4_l">
+      <dynamics damping="${joint_damping}"/>
+    </joint>
+    <link name="${name}_link_4_l">
       <inertial>
         <origin xyz="0 0 0" rpy="0 0 0"/>
@@ -425,5 +389,5 @@
       </collision>
     </link>
-   <!-- joint between link_4_l and link_5_l -->
+    <!-- joint between link_4_l and link_5_l -->
     <joint name="${name}_joint_4_l" type="revolute">
       <parent link="${name}_link_4_l"/>
@@ -433,11 +397,7 @@
       <limit lower="${-290 * PI / 180}" upper="${290 * PI / 180}"
              effort="${max_effort}" velocity="${400 * PI / 180}" />
-      <!--   <safety_controller soft_lower_limit="${-168 * M_PI / 180}"
-           soft_upper_limit="${168 * M_PI / 180}"
-           k_position="${safety_controller_k_pos}"
-           k_velocity="${safety_controller_k_vel}"/> -->
-      <dynamics damping="${joint_damping}"/>
-    </joint>
-   <link name="${name}_link_5_l">
+      <dynamics damping="${joint_damping}"/>
+    </joint>
+    <link name="${name}_link_5_l">
       <inertial>
         <origin xyz="0 0 0" rpy="0 0 0"/>
@@ -460,5 +420,5 @@
       </collision>
     </link>
-   <!-- joint between link_5_l and link_6_l -->
+    <!-- joint between link_5_l and link_6_l -->
     <joint name="${name}_joint_5_l" type="revolute">
       <parent link="${name}_link_5_l"/>
@@ -468,11 +428,7 @@
       <limit lower="${-88 * PI / 180}" upper="${138 * PI / 180}"
              effort="${max_effort}" velocity="${400 * PI / 180}" />
-      <!--   <safety_controller soft_lower_limit="${-168 * M_PI / 180}"
-           soft_upper_limit="${168 * M_PI / 180}"
-           k_position="${safety_controller_k_pos}"
-           k_velocity="${safety_controller_k_vel}"/> -->
-      <dynamics damping="${joint_damping}"/>
-    </joint>
-   <link name="${name}_link_6_l">
+      <dynamics damping="${joint_damping}"/>
+    </joint>
+    <link name="${name}_link_6_l">
       <inertial>
         <origin xyz="0 0 0" rpy="0 0 0"/>
@@ -495,5 +451,5 @@
       </collision>
     </link>
-   <!-- joint between link_6_l and link_7_l -->
+    <!-- joint between link_6_l and link_7_l -->
     <joint name="${name}_joint_6_l" type="revolute">
       <parent link="${name}_link_6_l"/>
@@ -503,11 +459,7 @@
       <limit lower="${-229 * PI / 180}" upper="${229 * PI / 180}"
              effort="${max_effort}" velocity="${400 * PI / 180}" />
-      <!--   <safety_controller soft_lower_limit="${-168 * M_PI / 180}"
-           soft_upper_limit="${168 * M_PI / 180}"
-           k_position="${safety_controller_k_pos}"
-           k_velocity="${safety_controller_k_vel}"/> -->
-      <dynamics damping="${joint_damping}"/>
-    </joint>
-   <link name="${name}_link_7_l">
+      <dynamics damping="${joint_damping}"/>
+    </joint>
+    <link name="${name}_link_7_l">
       <inertial>
         <origin xyz="0 0 0" rpy="0 0 0"/>

Commit message: Fixed grippers visualization bug.

File: yumi_description/urdf/yumi.xacro (robot description, xacro)
@@ -8,5 +8,5 @@
   <xacro:property name="joint_damping" value="0.5" />
   <xacro:property name="max_effort" value="300"/>
-  <xacro:macro name="yumi" params="name parent hardware_interface *origin">
+  <xacro:macro name="yumi" params="parent name hardware_interface *origin">
     <xacro:if value="${parent == 'world'}">
       <!--joint between world and body-->

Commit message: Fixed urdf

File: yumi_description/urdf/yumi.xacro (robot description, xacro)
@@ -276,5 +276,5 @@
           <mesh filename="package://yumi_description/meshes/link_7.stl"/>
         </geometry>
-        <material name="Blue"/>
+        <material name="Grey"/>
       </visual>
       <collision>
