Commit message: urdf seems to work

File: yumi_description/urdf/yumi.urdf.xacro (robot description, xacro)
@@ -3,6 +3,10 @@
   <!-- Import Rviz colors -->
   <xacro:include filename="$(find yumi_description)/urdf/materials.xacro" />
-  <!--Import the lbr iiwa macro -->
+  <!-- Import utilities -->
+  <xacro:include filename="$(find yumi_description)/urdf/utilities.xacro" />
+  <!--Import the yumi macro -->
   <xacro:include filename="$(find yumi_description)/urdf/yumi.xacro"/>
+  <!--Import the yumi servo gripper macro -->
+  <xacro:include filename="$(find yumi_description)/urdf/yumi_servo_gripper.xacro"/>
  <!-- Import Gazebo plugins -->
   <xacro:include filename="$(find yumi_description)/gazebo/gazebo.urdf.xacro"/>
@@ -13,3 +17,11 @@
     <origin xyz="0 0 0.1" rpy="0 0 0" />
   </xacro:yumi>
+  <!--right gripper-->
+  <xacro:yumi_servo_gripper name="gripper_r" hardware_interface="$(arg prefix)" parent="yumi_link_7_r">
+    <origin xyz="0 0 0.007" rpy="0 0 ${PI}" />
+  </xacro:yumi_servo_gripper>
+  <!--left gripper-->
+  <xacro:yumi_servo_gripper name="gripper_l" hardware_interface="$(arg prefix)" parent="yumi_link_7_l">
+    <origin xyz="0 0 0.007" rpy="0 0 ${PI}" />
+  </xacro:yumi_servo_gripper>
 </robot>

File: yumi_description/urdf/yumi.xacro (robot description, xacro)
@@ -40,4 +40,5 @@
       </collision>
     </link>
+   <!--///////////////////////////////////// RIGHT ARM ////////////////////////////////  -->
    <!-- joint between body and link_1_r -->
     <joint name="${name}_joint_1_r" type="revolute">
@@ -79,5 +80,5 @@
       <parent link="${name}_link_1_r"/>
       <child link="${name}_link_2_r"/>
-      <origin xyz="0.03 0.0 0.1" rpy="1.5708 0.0 0.0"/>
+      <origin xyz="0.03 0.0 0.1" rpy="${PI / 2} 0.0 0.0"/>
       <axis xyz="0 0 1"/>
       <limit lower="${-143.5 * PI / 180}" upper="${43.5 * PI / 180}"
@@ -111,8 +112,8 @@
     </link>
    <!-- joint between link_2_r and link_3_r -->
-    <joint name="${name}_joint_3_r" type="revolute">
+    <joint name="${name}_joint_7_r" type="revolute">
       <parent link="${name}_link_2_r"/>
       <child link="${name}_link_3_r"/>
-      <origin xyz="-0.03 0.17283 0.0" rpy="-1.5708 0.0 0.0"/>
+      <origin xyz="-0.03 0.17283 0.0" rpy="${-PI / 2} 0.0 0.0"/>
       <axis xyz="0 0 1"/>
       <limit lower="${-168.5 * PI / 180}" upper="${168.5 * PI / 180}"
@@ -146,8 +147,8 @@
     </link>
    <!-- joint between link_3_r and link_4_r -->
-    <joint name="${name}_joint_4_r" type="revolute">
+    <joint name="${name}_joint_3_r" type="revolute">
       <parent link="${name}_link_3_r"/>
       <child link="${name}_link_4_r"/>
-      <origin xyz="-0.04188 0.0 0.07873" rpy="1.5708 -1.5708 0.0"/>
+      <origin xyz="-0.04188 0.0 0.07873" rpy="${PI / 2} ${- PI / 2} 0.0"/>
       <axis xyz="0 0 1"/>
       <limit lower="${-123.5 * PI / 180}" upper="${80 * PI / 180}"
@@ -181,8 +182,8 @@
     </link>
    <!-- joint between link_4_r and link_5_r -->
-    <joint name="${name}_joint_5_r" type="revolute">
+    <joint name="${name}_joint_4_r" type="revolute">
       <parent link="${name}_link_4_r"/>
       <child link="${name}_link_5_r"/>
-      <origin xyz="0.0405 0.16461 0.0" rpy="-1.5708 0.0 0.0"/>
+      <origin xyz="0.0405 0.16461 0.0" rpy="-${PI / 2} 0.0 0.0"/>
       <axis xyz="0 0 1"/>
       <limit lower="${-290 * PI / 180}" upper="${290 * PI / 180}"
@@ -216,8 +217,8 @@
     </link>
    <!-- joint between link_5_r and link_6_r -->
-    <joint name="${name}_joint_6_r" type="revolute">
+    <joint name="${name}_joint_5_r" type="revolute">
       <parent link="${name}_link_5_r"/>
       <child link="${name}_link_6_r"/>
-      <origin xyz="-0.027 0 0.10039" rpy="1.5708 0.0 0.0"/>
+      <origin xyz="-0.027 0 0.10039" rpy="${PI / 2} 0.0 0.0"/>
       <axis xyz="0 0 1"/>
       <limit lower="${-88 * PI / 180}" upper="${138 * PI / 180}"
@@ -251,8 +252,8 @@
     </link>
    <!-- joint between link_6_r and link_7_r -->
-    <joint name="${name}_joint_7_r" type="revolute">
+    <joint name="${name}_joint_6_r" type="revolute">
       <parent link="${name}_link_6_r"/>
       <child link="${name}_link_7_r"/>
-      <origin xyz="0.027 0.029 0.0" rpy="-1.5708 0.0 0.0"/>
+      <origin xyz="0.027 0.029 0.0" rpy="-${PI / 2} 0.0 0.0"/>
       <axis xyz="0 0 1"/>
       <limit lower="${-229 * PI / 180}" upper="${229 * PI / 180}"
@@ -265,4 +266,250 @@
     </joint>
    <link name="${name}_link_7_r">
+      <inertial>
+        <origin xyz="0 0 0" rpy="0 0 0"/>
+        <mass value="2"/>
+        <inertia ixx="0.1"  ixy="0"  ixz="0" iyy="0.1" iyz="0" izz="0.1" />
+      </inertial>
+      <visual>
+        <origin xyz="0 0 0" rpy="0 0 0"/>
+        <geometry>
+          <mesh filename="package://yumi_description/meshes/link_7.stl"/>
+        </geometry>
+        <material name="Grey"/>
+      </visual>
+      <collision>
+        <origin xyz="0 0 0" rpy="0 0 0"/>
+        <geometry>
+          <mesh filename="package://yumi_description/meshes/coarse/link_7.stl"/>
+        </geometry>
+        <material name="Grey"/>
+      </collision>
+    </link>
+   <!--///////////////////////////////////// LEFT ARM ////////////////////////////////  -->
+  <!-- joint between body and link_1_l -->
+    <joint name="${name}_joint_1_l" type="revolute">
+      <parent link="${name}_body"/>
+      <child link="${name}_link_1_l"/>
+      <origin xyz="0.05355 0.07250 0.41492" rpy="0.9781 -0.5716 2.3180"/>
+      <axis xyz="0 0 1"/>
+      <limit lower="${-168.5 * PI / 180}" upper="${168.5 * PI / 180}"
+             effort="${max_effort}" velocity="${180 * PI / 180}" />
+      <!--   <safety_controller soft_lower_limit="${-168 * M_PI / 180}"
+           soft_upper_limit="${168 * M_PI / 180}"
+           k_position="${safety_controller_k_pos}"
+           k_velocity="${safety_controller_k_vel}"/> -->
+      <dynamics damping="${joint_damping}"/>
+    </joint>
+   <link name="${name}_link_1_l">
+      <inertial>
+        <origin xyz="0 -0.03 0.12" rpy="0 0 0"/>
+        <mass value="2"/>
+        <inertia ixx="0.1"  ixy="0"  ixz="0" iyy="0.1" iyz="0" izz="0.1" />
+      </inertial>
+      <visual>
+        <origin xyz="0 0 0" rpy="0 0 0"/>
+        <geometry>
+          <mesh filename="package://yumi_description/meshes/link_1.stl"/>
+        </geometry>
+        <material name="Grey"/>
+      </visual>
+      <collision>
+        <origin xyz="0 0 0" rpy="0 0 0"/>
+        <geometry>
+          <mesh filename="package://yumi_description/meshes/coarse/link_1.stl"/>
+        </geometry>
+        <material name="Grey"/>
+      </collision>
+    </link>
+ <!-- joint between link_1_l and link_2_l -->
+    <joint name="${name}_joint_2_l" type="revolute">
+      <parent link="${name}_link_1_l"/>
+      <child link="${name}_link_2_l"/>
+      <origin xyz="0.03 0.0 0.1" rpy="${PI / 2} 0.0 0.0"/>
+      <axis xyz="0 0 1"/>
+      <limit lower="${-143.5 * PI / 180}" upper="${43.5 * PI / 180}"
+             effort="${max_effort}" velocity="${180 * PI / 180}" />
+      <!--   <safety_controller soft_lower_limit="${-168 * M_PI / 180}"
+           soft_upper_limit="${168 * M_PI / 180}"
+           k_position="${safety_controller_k_pos}"
+           k_velocity="${safety_controller_k_vel}"/> -->
+      <dynamics damping="${joint_damping}"/>
+    </joint>
+   <link name="${name}_link_2_l">
+      <inertial>
+        <origin xyz="0 0 0" rpy="0 0 0"/>
+        <mass value="2"/>
+        <inertia ixx="0.1"  ixy="0"  ixz="0" iyy="0.1" iyz="0" izz="0.1" />
+      </inertial>
+      <visual>
+        <origin xyz="0 0 0" rpy="0 0 0"/>
+        <geometry>
+          <mesh filename="package://yumi_description/meshes/link_2.stl"/>
+        </geometry>
+        <material name="Grey"/>
+      </visual>
+      <collision>
+        <origin xyz="0 0 0" rpy="0 0 0"/>
+        <geometry>
+          <mesh filename="package://yumi_description/meshes/coarse/link_2.stl"/>
+        </geometry>
+        <material name="Grey"/>
+      </collision>
+    </link>
+ <!-- joint between link_2_l and link_3_l -->
+    <joint name="${name}_joint_7_l" type="revolute">
+      <parent link="${name}_link_2_l"/>
+      <child link="${name}_link_3_l"/>
+      <origin xyz="-0.03 0.17283 0.0" rpy="-${PI / 2} 0.0 0.0"/>
+      <axis xyz="0 0 1"/>
+      <limit lower="${-168.5 * PI / 180}" upper="${168.5 * PI / 180}"
+             effort="${max_effort}" velocity="${180 * PI / 180}" />
+      <!--   <safety_controller soft_lower_limit="${-168 * M_PI / 180}"
+           soft_upper_limit="${168 * M_PI / 180}"
+           k_position="${safety_controller_k_pos}"
+           k_velocity="${safety_controller_k_vel}"/> -->
+      <dynamics damping="${joint_damping}"/>
+    </joint>
+   <link name="${name}_link_3_l">
+      <inertial>
+        <origin xyz="0 0 0" rpy="0 0 0"/>
+        <mass value="2"/>
+        <inertia ixx="0.1"  ixy="0"  ixz="0" iyy="0.1" iyz="0" izz="0.1" />
+      </inertial>
+      <visual>
+        <origin xyz="0 0 0" rpy="0 0 0"/>
+        <geometry>
+          <mesh filename="package://yumi_description/meshes/link_3.stl"/>
+        </geometry>
+        <material name="Grey"/>
+      </visual>
+      <collision>
+        <origin xyz="0 0 0" rpy="0 0 0"/>
+        <geometry>
+          <mesh filename="package://yumi_description/meshes/coarse/link_3.stl"/>
+        </geometry>
+        <material name="Grey"/>
+      </collision>
+    </link>
+   <!-- joint between link_3_l and link_4_l -->
+    <joint name="${name}_joint_3_l" type="revolute">
+      <parent link="${name}_link_3_l"/>
+      <child link="${name}_link_4_l"/>
+      <origin xyz="-0.04188 0.0 0.07873" rpy="${PI / 2} -${PI / 2} 0.0"/>
+      <axis xyz="0 0 1"/>
+      <limit lower="${-123.5 * PI / 180}" upper="${80 * PI / 180}"
+             effort="${max_effort}" velocity="${180 * PI / 180}" />
+      <!--   <safety_controller soft_lower_limit="${-168 * M_PI / 180}"
+           soft_upper_limit="${168 * M_PI / 180}"
+           k_position="${safety_controller_k_pos}"
+           k_velocity="${safety_controller_k_vel}"/> -->
+      <dynamics damping="${joint_damping}"/>
+    </joint>
+   <link name="${name}_link_4_l">
+      <inertial>
+        <origin xyz="0 0 0" rpy="0 0 0"/>
+        <mass value="2"/>
+        <inertia ixx="0.1"  ixy="0"  ixz="0" iyy="0.1" iyz="0" izz="0.1" />
+      </inertial>
+      <visual>
+        <origin xyz="0 0 0" rpy="0 0 0"/>
+        <geometry>
+          <mesh filename="package://yumi_description/meshes/link_4.stl"/>
+        </geometry>
+        <material name="Grey"/>
+      </visual>
+      <collision>
+        <origin xyz="0 0 0" rpy="0 0 0"/>
+        <geometry>
+          <mesh filename="package://yumi_description/meshes/coarse/link_4.stl"/>
+        </geometry>
+        <material name="Grey"/>
+      </collision>
+    </link>
+   <!-- joint between link_4_l and link_5_l -->
+    <joint name="${name}_joint_4_l" type="revolute">
+      <parent link="${name}_link_4_l"/>
+      <child link="${name}_link_5_l"/>
+      <origin xyz="0.0405 0.16461 0.0" rpy="-${PI / 2} 0.0 0.0"/>
+      <axis xyz="0 0 1"/>
+      <limit lower="${-290 * PI / 180}" upper="${290 * PI / 180}"
+             effort="${max_effort}" velocity="${400 * PI / 180}" />
+      <!--   <safety_controller soft_lower_limit="${-168 * M_PI / 180}"
+           soft_upper_limit="${168 * M_PI / 180}"
+           k_position="${safety_controller_k_pos}"
+           k_velocity="${safety_controller_k_vel}"/> -->
+      <dynamics damping="${joint_damping}"/>
+    </joint>
+   <link name="${name}_link_5_l">
+      <inertial>
+        <origin xyz="0 0 0" rpy="0 0 0"/>
+        <mass value="2"/>
+        <inertia ixx="0.1"  ixy="0"  ixz="0" iyy="0.1" iyz="0" izz="0.1" />
+      </inertial>
+      <visual>
+        <origin xyz="0 0 0" rpy="0 0 0"/>
+        <geometry>
+          <mesh filename="package://yumi_description/meshes/link_5.stl"/>
+        </geometry>
+        <material name="Grey"/>
+      </visual>
+      <collision>
+        <origin xyz="0 0 0" rpy="0 0 0"/>
+        <geometry>
+          <mesh filename="package://yumi_description/meshes/coarse/link_5.stl"/>
+        </geometry>
+        <material name="Grey"/>
+      </collision>
+    </link>
+   <!-- joint between link_5_l and link_6_l -->
+    <joint name="${name}_joint_5_l" type="revolute">
+      <parent link="${name}_link_5_l"/>
+      <child link="${name}_link_6_l"/>
+      <origin xyz="-0.027 0 0.10039" rpy="${PI / 2} 0.0 0.0"/>
+      <axis xyz="0 0 1"/>
+      <limit lower="${-88 * PI / 180}" upper="${138 * PI / 180}"
+             effort="${max_effort}" velocity="${400 * PI / 180}" />
+      <!--   <safety_controller soft_lower_limit="${-168 * M_PI / 180}"
+           soft_upper_limit="${168 * M_PI / 180}"
+           k_position="${safety_controller_k_pos}"
+           k_velocity="${safety_controller_k_vel}"/> -->
+      <dynamics damping="${joint_damping}"/>
+    </joint>
+   <link name="${name}_link_6_l">
+      <inertial>
+        <origin xyz="0 0 0" rpy="0 0 0"/>
+        <mass value="2"/>
+        <inertia ixx="0.1"  ixy="0"  ixz="0" iyy="0.1" iyz="0" izz="0.1" />
+      </inertial>
+      <visual>
+        <origin xyz="0 0 0" rpy="0 0 0"/>
+        <geometry>
+          <mesh filename="package://yumi_description/meshes/link_6.stl"/>
+        </geometry>
+        <material name="Grey"/>
+      </visual>
+      <collision>
+        <origin xyz="0 0 0" rpy="0 0 0"/>
+        <geometry>
+          <mesh filename="package://yumi_description/meshes/coarse/link_6.stl"/>
+        </geometry>
+        <material name="Grey"/>
+      </collision>
+    </link>
+   <!-- joint between link_6_l and link_7_l -->
+    <joint name="${name}_joint_6_l" type="revolute">
+      <parent link="${name}_link_6_l"/>
+      <child link="${name}_link_7_l"/>
+      <origin xyz="0.027 0.029 0.0" rpy="${-PI / 2} 0.0 0.0"/>
+      <axis xyz="0 0 1"/>
+      <limit lower="${-229 * PI / 180}" upper="${229 * PI / 180}"
+             effort="${max_effort}" velocity="${400 * PI / 180}" />
+      <!--   <safety_controller soft_lower_limit="${-168 * M_PI / 180}"
+           soft_upper_limit="${168 * M_PI / 180}"
+           k_position="${safety_controller_k_pos}"
+           k_velocity="${safety_controller_k_vel}"/> -->
+      <dynamics damping="${joint_damping}"/>
+    </joint>
+   <link name="${name}_link_7_l">
       <inertial>
         <origin xyz="0 0 0" rpy="0 0 0"/>

Commit message: Changed the grippers interface to EffortJointInterface in the URDF. Deleted all grippers rws file. Updated the general launch files

File: yumi_description/urdf/yumi.urdf.xacro (robot description, xacro)
@@ -14,13 +14,13 @@
   <link name="world"/>
   <!--yumi-->
-  <xacro:yumi name="yumi" hardware_interface="$(arg prefix)" parent="world">
+  <xacro:yumi name="yumi" hardware_interface="hardware_interface/$(arg prefix)" parent="world">
     <origin xyz="0 0 0.1" rpy="0 0 0" />
   </xacro:yumi>
   <!--right gripper-->
-  <xacro:yumi_servo_gripper name="gripper_r" hardware_interface="$(arg prefix)" parent="yumi_link_7_r">
+  <xacro:yumi_servo_gripper name="gripper_r" hardware_interface="hardware_interface/EffortJointInterface" parent="yumi_link_7_r">
     <origin xyz="0 0 0.007" rpy="0 0 ${PI}" />
   </xacro:yumi_servo_gripper>
   <!--left gripper-->
-  <xacro:yumi_servo_gripper name="gripper_l" hardware_interface="$(arg prefix)" parent="yumi_link_7_l">
+  <xacro:yumi_servo_gripper name="gripper_l" hardware_interface="hardware_interface/EffortJointInterface" parent="yumi_link_7_l">
     <origin xyz="0 0 0.007" rpy="0 0 ${PI}" />
   </xacro:yumi_servo_gripper>

File: yumi_description/urdf/yumi_servo_gripper.xacro (robot description, xacro)
@@ -1,15 +1,15 @@
 <?xml version="1.0"?>
 <robot name="yumi" xmlns:xacro="http://www.ros.org/wiki/xacro">
-  <!-- Import all Gazebo-customization elements, including Gazebo colors -->
-  <xacro:include filename="$(find yumi_description)/urdf/yumi_servo_gripper.gazebo.xacro" />
-  <!-- Import Transmissions -->
-  <xacro:include filename="$(find yumi_description)/urdf/yumi_servo_gripper.transmission.xacro" />
-  <!-- Include Utilities -->
-  <xacro:include filename="$(find yumi_description)/urdf/utilities.xacro" />
-  <!-- some constants -->
- <!-- <xacro:property name="safety_controller_k_pos" value="100" />
-  <xacro:property name="safety_controller_k_vel" value="2" /> -->
-  <xacro:property name="joint_damping" value="0.5" />
-  <xacro:property name="max_effort" value="300"/>
+    <!-- Import all Gazebo-customization elements, including Gazebo colors -->
+    <xacro:include filename="$(find yumi_description)/urdf/yumi_servo_gripper.gazebo.xacro" />
+    <!-- Import Transmissions -->
+    <xacro:include filename="$(find yumi_description)/urdf/yumi_servo_gripper.transmission.xacro" />
+    <!-- Include Utilities -->
+    <xacro:include filename="$(find yumi_description)/urdf/utilities.xacro" />
+    <!-- some constants -->
+    <xacro:property name="joint_damping" value="0.5" />
+    <xacro:property name="gripper_joint_damping" value="1.0" />
+    <xacro:property name="max_gripper_effort" value="50"/>
+    <xacro:property name="max_gripper_velocity" value="2"/>
   <xacro:macro name="yumi_servo_gripper" params="parent name hardware_interface *origin">
     <!--joint between {parent} and base-->
@@ -47,10 +47,10 @@
       <axis xyz="-1 0 0"/>
       <limit lower="0" upper="0.025"
-             effort="${max_effort}" velocity="0.02" />
+             effort="${max_gripper_effort}" velocity="${max_gripper_velocity}" />
       <!--   <safety_controller soft_lower_limit="${-168 * M_PI / 180}"
            soft_upper_limit="${168 * M_PI / 180}"
            k_position="${safety_controller_k_pos}"
            k_velocity="${safety_controller_k_vel}"/> -->
-      <dynamics damping="${joint_damping}"/>
+      <dynamics damping="${gripper_joint_damping}"/>
     </joint>
     <link name="${name}_finger_r">
@@ -65,5 +65,5 @@
           <mesh filename="package://yumi_description/meshes/gripper/finger.stl"/>
         </geometry>
-        <material name="Grey"/>
+        <material name="Blue"/>
       </visual>
       <collision>
@@ -72,5 +72,5 @@
           <mesh filename="package://yumi_description/meshes/gripper/coarse/finger.stl"/>
         </geometry>
-        <material name="Grey"/>
+        <material name="Blue"/>
       </collision>
     </link>
@@ -82,10 +82,10 @@
       <axis xyz="-1 0 0"/>
       <limit lower="0" upper="0.025"
-             effort="${max_effort}" velocity="0.02" />
+             effort="${max_gripper_effort}" velocity="${max_gripper_velocity}" />
       <!--   <safety_controller soft_lower_limit="${-168 * M_PI / 180}"
            soft_upper_limit="${168 * M_PI / 180}"
            k_position="${safety_controller_k_pos}"
            k_velocity="${safety_controller_k_vel}"/> -->
-      <dynamics damping="${joint_damping}"/>
+      <dynamics damping="${gripper_joint_damping}"/>
       <mimic joint="${name}_joint"/>
     </joint>
@@ -101,5 +101,5 @@
           <mesh filename="package://yumi_description/meshes/gripper/finger.stl"/>
         </geometry>
-        <material name="Grey"/>
+        <material name="Blue"/>
       </visual>
       <collision>
@@ -108,5 +108,5 @@
           <mesh filename="package://yumi_description/meshes/gripper/coarse/finger.stl"/>
         </geometry>
-        <material name="Grey"/>
+        <material name="Blue"/>
       </collision>
     </link>
