Commit message: Revert "Merge pull request #13 from kth-ros-pkg/egm_modifications"  revertin merge into master. PR is now in branch feature-egm (hopefully)
This reverts commit e3b71a8f4bf1f8e69048eff7e7b5b6f3f5491120, reversing
changes made to f4a6680138c808bed64ddcd5b7b29aa4d5398ad7.

File: yumi_description/urdf/yumi.urdf.xacro (robot description, xacro)
@@ -2,25 +2,25 @@
 <robot name="yumi" xmlns:xacro="http://www.ros.org/wiki/xacro">
   <!-- Import Rviz colors -->
-  <xacro:include filename="$(find yumi_description)/urdf/Util/materials.xacro" />
+  <xacro:include filename="$(find yumi_description)/urdf/materials.xacro" />
   <!-- Import utilities -->
-  <xacro:include filename="$(find yumi_description)/urdf/Util/utilities.xacro" />
+  <xacro:include filename="$(find yumi_description)/urdf/utilities.xacro" />
   <!--Import the yumi macro -->
   <xacro:include filename="$(find yumi_description)/urdf/yumi.xacro"/>
   <!--Import the yumi servo gripper macro -->
-  <xacro:include filename="$(find yumi_description)/urdf/Grippers/yumi_servo_gripper.xacro"/>
-  <!-- Import Gazebo plugins -->
-  <xacro:include filename="$(find yumi_description)/urdf/Gazebo/gazebo.urdf.xacro"/>
+  <xacro:include filename="$(find yumi_description)/urdf/yumi_servo_gripper.xacro"/>
+ <!-- Import Gazebo plugins -->
+  <xacro:include filename="$(find yumi_description)/gazebo/gazebo.urdf.xacro"/>
   <!-- Fix to world just for testing -->
   <link name="world"/>
   <!--yumi-->
-  <xacro:yumi name="yumi" hardware_interface="hardware_interface/$(arg arms_interface)" parent="world">
+  <xacro:yumi name="yumi" hardware_interface="$(arg prefix)" parent="world">
     <origin xyz="0 0 0.1" rpy="0 0 0" />
   </xacro:yumi>
   <!--right gripper-->
-  <xacro:yumi_servo_gripper name="gripper_r" hardware_interface="hardware_interface/$(arg grippers_interface)" parent="yumi_link_7_r">
+  <xacro:yumi_servo_gripper name="gripper_r" hardware_interface="$(arg prefix)" parent="yumi_link_7_r">
     <origin xyz="0 0 0.007" rpy="0 0 ${PI}" />
   </xacro:yumi_servo_gripper>
   <!--left gripper-->
-  <xacro:yumi_servo_gripper name="gripper_l" hardware_interface="hardware_interface/$(arg grippers_interface)" parent="yumi_link_7_l">
+  <xacro:yumi_servo_gripper name="gripper_l" hardware_interface="$(arg prefix)" parent="yumi_link_7_l">
     <origin xyz="0 0 0.007" rpy="0 0 ${PI}" />
   </xacro:yumi_servo_gripper>

File: yumi_description/urdf/yumi.xacro (robot description, xacro)
@@ -2,19 +2,21 @@
 <robot name="yumi" xmlns:xacro="http://www.ros.org/wiki/xacro">
   <!-- Import all Gazebo-customization elements, including Gazebo colors -->
-  <xacro:include filename="$(find yumi_description)/urdf/Gazebo/yumi.gazebo.xacro" />
+  <xacro:include filename="$(find yumi_description)/urdf/yumi.gazebo.xacro" />
   <!-- Import Transmissions -->
   <xacro:include filename="$(find yumi_description)/urdf/yumi.transmission.xacro" />
+  <!-- Include Utilities -->
+  <xacro:include filename="$(find yumi_description)/urdf/utilities.xacro" />
   <!-- some constants -->
+ <!-- <xacro:property name="safety_controller_k_pos" value="100" />
+  <xacro:property name="safety_controller_k_vel" value="2" /> -->
   <xacro:property name="joint_damping" value="0.5" />
   <xacro:property name="max_effort" value="300"/>
-  <xacro:macro name="yumi" params="name parent hardware_interface *origin">
-    <xacro:if value="${parent == 'world'}">
-      <!--joint between world and body-->
-      <joint name="world_joint" type="fixed">
-        <insert_block name="origin"/>
-        <parent link="world"/>
-        <child link="${name}_body"/>
-      </joint>
-    </xacro:if>
+  <xacro:macro name="yumi" params="parent name hardware_interface *origin">
+    <!--joint between {parent} and body-->
+    <joint name="${parent}_joint" type="fixed">
+      <insert_block name="origin"/>
+      <parent link="${parent}"/>
+      <child link="${name}_body"/>
+    </joint>
     <link name="${name}_body">
       <inertial>
@@ -47,4 +49,8 @@
       <limit lower="${-168.5 * PI / 180}" upper="${168.5 * PI / 180}"
              effort="${max_effort}" velocity="${180 * PI / 180}" />
+      <!--   <safety_controller soft_lower_limit="${-168 * M_PI / 180}"
+           soft_upper_limit="${168 * M_PI / 180}"
+           k_position="${safety_controller_k_pos}"
+           k_velocity="${safety_controller_k_vel}"/> -->
       <dynamics damping="${joint_damping}"/>
     </joint>
@@ -78,7 +84,11 @@
       <limit lower="${-143.5 * PI / 180}" upper="${43.5 * PI / 180}"
              effort="${max_effort}" velocity="${180 * PI / 180}" />
-      <dynamics damping="${joint_damping}"/>
-    </joint>
-    <link name="${name}_link_2_r">
+      <!--   <safety_controller soft_lower_limit="${-168 * M_PI / 180}"
+           soft_upper_limit="${168 * M_PI / 180}"
+           k_position="${safety_controller_k_pos}"
+           k_velocity="${safety_controller_k_vel}"/> -->
+      <dynamics damping="${joint_damping}"/>
+    </joint>
+   <link name="${name}_link_2_r">
       <inertial>
         <origin xyz="0 0 0" rpy="0 0 0"/>
@@ -101,15 +111,19 @@
       </collision>
     </link>
-     <!-- joint between link_2_r and link_3_r -->
-      <joint name="${name}_joint_7_r" type="revolute">
-        <parent link="${name}_link_2_r"/>
-        <child link="${name}_link_3_r"/>
-        <origin xyz="-0.03 0.17283 0.0" rpy="${-PI / 2} 0.0 0.0"/>
-        <axis xyz="0 0 1"/>
-        <limit lower="${-168.5 * PI / 180}" upper="${168.5 * PI / 180}"
-               effort="${max_effort}" velocity="${180 * PI / 180}" />
-        <dynamics damping="${joint_damping}"/>
-      </joint>
-    <link name="${name}_link_3_r">
+   <!-- joint between link_2_r and link_3_r -->
+    <joint name="${name}_joint_7_r" type="revolute">
+      <parent link="${name}_link_2_r"/>
+      <child link="${name}_link_3_r"/>
+      <origin xyz="-0.03 0.17283 0.0" rpy="${-PI / 2} 0.0 0.0"/>
+      <axis xyz="0 0 1"/>
+      <limit lower="${-168.5 * PI / 180}" upper="${168.5 * PI / 180}"
+             effort="${max_effort}" velocity="${180 * PI / 180}" />
+      <!--   <safety_controller soft_lower_limit="${-168 * M_PI / 180}"
+           soft_upper_limit="${168 * M_PI / 180}"
+           k_position="${safety_controller_k_pos}"
+           k_velocity="${safety_controller_k_vel}"/> -->
+      <dynamics damping="${joint_damping}"/>
+    </joint>
+   <link name="${name}_link_3_r">
       <inertial>
         <origin xyz="0 0 0" rpy="0 0 0"/>
@@ -132,5 +146,5 @@
       </collision>
     </link>
-    <!-- joint between link_3_r and link_4_r -->
+   <!-- joint between link_3_r and link_4_r -->
     <joint name="${name}_joint_3_r" type="revolute">
       <parent link="${name}_link_3_r"/>
@@ -140,7 +154,11 @@
       <limit lower="${-123.5 * PI / 180}" upper="${80 * PI / 180}"
              effort="${max_effort}" velocity="${180 * PI / 180}" />
-      <dynamics damping="${joint_damping}"/>
-    </joint>
-    <link name="${name}_link_4_r">
+      <!--   <safety_controller soft_lower_limit="${-168 * M_PI / 180}"
+           soft_upper_limit="${168 * M_PI / 180}"
+           k_position="${safety_controller_k_pos}"
+           k_velocity="${safety_controller_k_vel}"/> -->
+      <dynamics damping="${joint_damping}"/>
+    </joint>
+   <link name="${name}_link_4_r">
       <inertial>
         <origin xyz="0 0 0" rpy="0 0 0"/>
@@ -163,5 +181,5 @@
       </collision>
     </link>
-    <!-- joint between link_4_r and link_5_r -->
+   <!-- joint between link_4_r and link_5_r -->
     <joint name="${name}_joint_4_r" type="revolute">
       <parent link="${name}_link_4_r"/>
@@ -171,7 +189,11 @@
       <limit lower="${-290 * PI / 180}" upper="${290 * PI / 180}"
              effort="${max_effort}" velocity="${400 * PI / 180}" />
-      <dynamics damping="${joint_damping}"/>
-    </joint>
-    <link name="${name}_link_5_r">
+      <!--   <safety_controller soft_lower_limit="${-168 * M_PI / 180}"
+           soft_upper_limit="${168 * M_PI / 180}"
+           k_position="${safety_controller_k_pos}"
+           k_velocity="${safety_controller_k_vel}"/> -->
+      <dynamics damping="${joint_damping}"/>
+    </joint>
+   <link name="${name}_link_5_r">
       <inertial>
         <origin xyz="0 0 0" rpy="0 0 0"/>
@@ -194,5 +216,5 @@
       </collision>
     </link>
-    <!-- joint between link_5_r and link_6_r -->
+   <!-- joint between link_5_r and link_6_r -->
     <joint name="${name}_joint_5_r" type="revolute">
       <parent link="${name}_link_5_r"/>
@@ -202,7 +224,11 @@
       <limit lower="${-88 * PI / 180}" upper="${138 * PI / 180}"
              effort="${max_effort}" velocity="${400 * PI / 180}" />
-      <dynamics damping="${joint_damping}"/>
-    </joint>
-    <link name="${name}_link_6_r">
+      <!--   <safety_controller soft_lower_limit="${-168 * M_PI / 180}"
+           soft_upper_limit="${168 * M_PI / 180}"
+           k_position="${safety_controller_k_pos}"
+           k_velocity="${safety_controller_k_vel}"/> -->
+      <dynamics damping="${joint_damping}"/>
+    </joint>
+   <link name="${name}_link_6_r">
       <inertial>
         <origin xyz="0 0 0" rpy="0 0 0"/>
@@ -225,5 +251,5 @@
       </collision>
     </link>
-    <!-- joint between link_6_r and link_7_r -->
+   <!-- joint between link_6_r and link_7_r -->
     <joint name="${name}_joint_6_r" type="revolute">
       <parent link="${name}_link_6_r"/>
@@ -233,7 +259,11 @@
       <limit lower="${-229 * PI / 180}" upper="${229 * PI / 180}"
              effort="${max_effort}" velocity="${400 * PI / 180}" />
-      <dynamics damping="${joint_damping}"/>
-    </joint>
-    <link name="${name}_link_7_r">
+      <!--   <safety_controller soft_lower_limit="${-168 * M_PI / 180}"
+           soft_upper_limit="${168 * M_PI / 180}"
+           k_position="${safety_controller_k_pos}"
+           k_velocity="${safety_controller_k_vel}"/> -->
+      <dynamics damping="${joint_damping}"/>
+    </joint>
+   <link name="${name}_link_7_r">
       <inertial>
         <origin xyz="0 0 0" rpy="0 0 0"/>
@@ -256,6 +286,6 @@
       </collision>
     </link>
-    <!--///////////////////////////////////// LEFT ARM ////////////////////////////////  -->
-    <!-- joint between body and link_1_l -->
+   <!--///////////////////////////////////// LEFT ARM ////////////////////////////////  -->
+  <!-- joint between body and link_1_l -->
     <joint name="${name}_joint_1_l" type="revolute">
       <parent link="${name}_body"/>
@@ -265,7 +295,11 @@
       <limit lower="${-168.5 * PI / 180}" upper="${168.5 * PI / 180}"
              effort="${max_effort}" velocity="${180 * PI / 180}" />
-      <dynamics damping="${joint_damping}"/>
-    </joint>
-    <link name="${name}_link_1_l">
+      <!--   <safety_controller soft_lower_limit="${-168 * M_PI / 180}"
+           soft_upper_limit="${168 * M_PI / 180}"
+           k_position="${safety_controller_k_pos}"
+           k_velocity="${safety_controller_k_vel}"/> -->
+      <dynamics damping="${joint_damping}"/>
+    </joint>
+   <link name="${name}_link_1_l">
       <inertial>
         <origin xyz="0 -0.03 0.12" rpy="0 0 0"/>
@@ -288,5 +322,5 @@
       </collision>
     </link>
-    <!-- joint between link_1_l and link_2_l -->
+ <!-- joint between link_1_l and link_2_l -->
     <joint name="${name}_joint_2_l" type="revolute">
       <parent link="${name}_link_1_l"/>
@@ -296,7 +330,11 @@
       <limit lower="${-143.5 * PI / 180}" upper="${43.5 * PI / 180}"
              effort="${max_effort}" velocity="${180 * PI / 180}" />
-      <dynamics damping="${joint_damping}"/>
-    </joint>
-    <link name="${name}_link_2_l">
+      <!--   <safety_controller soft_lower_limit="${-168 * M_PI / 180}"
+           soft_upper_limit="${168 * M_PI / 180}"
+           k_position="${safety_controller_k_pos}"
+           k_velocity="${safety_controller_k_vel}"/> -->
+      <dynamics damping="${joint_damping}"/>
+    </joint>
+   <link name="${name}_link_2_l">
       <inertial>
         <origin xyz="0 0 0" rpy="0 0 0"/>
@@ -319,5 +357,5 @@
       </collision>
     </link>
-    <!-- joint between link_2_l and link_3_l -->
+ <!-- joint between link_2_l and link_3_l -->
     <joint name="${name}_joint_7_l" type="revolute">
       <parent link="${name}_link_2_l"/>
@@ -327,7 +365,11 @@
       <limit lower="${-168.5 * PI / 180}" upper="${168.5 * PI / 180}"
              effort="${max_effort}" velocity="${180 * PI / 180}" />
-      <dynamics damping="${joint_damping}"/>
-    </joint>
-    <link name="${name}_link_3_l">
+      <!--   <safety_controller soft_lower_limit="${-168 * M_PI / 180}"
+           soft_upper_limit="${168 * M_PI / 180}"
+           k_position="${safety_controller_k_pos}"
+           k_velocity="${safety_controller_k_vel}"/> -->
+      <dynamics damping="${joint_damping}"/>
+    </joint>
+   <link name="${name}_link_3_l">
       <inertial>
         <origin xyz="0 0 0" rpy="0 0 0"/>
@@ -350,5 +392,5 @@
       </collision>
     </link>
-    <!-- joint between link_3_l and link_4_l -->
+   <!-- joint between link_3_l and link_4_l -->
     <joint name="${name}_joint_3_l" type="revolute">
       <parent link="${name}_link_3_l"/>
@@ -358,7 +400,11 @@
       <limit lower="${-123.5 * PI / 180}" upper="${80 * PI / 180}"
              effort="${max_effort}" velocity="${180 * PI / 180}" />
-      <dynamics damping="${joint_damping}"/>
-    </joint>
-    <link name="${name}_link_4_l">
+      <!--   <safety_controller soft_lower_limit="${-168 * M_PI / 180}"
+           soft_upper_limit="${168 * M_PI / 180}"
+           k_position="${safety_controller_k_pos}"
+           k_velocity="${safety_controller_k_vel}"/> -->
+      <dynamics damping="${joint_damping}"/>
+    </joint>
+   <link name="${name}_link_4_l">
       <inertial>
         <origin xyz="0 0 0" rpy="0 0 0"/>
@@ -381,5 +427,5 @@
       </collision>
     </link>
-    <!-- joint between link_4_l and link_5_l -->
+   <!-- joint between link_4_l and link_5_l -->
     <joint name="${name}_joint_4_l" type="revolute">
       <parent link="${name}_link_4_l"/>
@@ -389,7 +435,11 @@
       <limit lower="${-290 * PI / 180}" upper="${290 * PI / 180}"
              effort="${max_effort}" velocity="${400 * PI / 180}" />
-      <dynamics damping="${joint_damping}"/>
-    </joint>
-    <link name="${name}_link_5_l">
+      <!--   <safety_controller soft_lower_limit="${-168 * M_PI / 180}"
+           soft_upper_limit="${168 * M_PI / 180}"
+           k_position="${safety_controller_k_pos}"
+           k_velocity="${safety_controller_k_vel}"/> -->
+      <dynamics damping="${joint_damping}"/>
+    </joint>
+   <link name="${name}_link_5_l">
       <inertial>
         <origin xyz="0 0 0" rpy="0 0 0"/>
@@ -412,5 +462,5 @@
       </collision>
     </link>
-    <!-- joint between link_5_l and link_6_l -->
+   <!-- joint between link_5_l and link_6_l -->
     <joint name="${name}_joint_5_l" type="revolute">
       <parent link="${name}_link_5_l"/>
@@ -420,7 +470,11 @@
       <limit lower="${-88 * PI / 180}" upper="${138 * PI / 180}"
              effort="${max_effort}" velocity="${400 * PI / 180}" />
-      <dynamics damping="${joint_damping}"/>
-    </joint>
-    <link name="${name}_link_6_l">
+      <!--   <safety_controller soft_lower_limit="${-168 * M_PI / 180}"
+           soft_upper_limit="${168 * M_PI / 180}"
+           k_position="${safety_controller_k_pos}"
+           k_velocity="${safety_controller_k_vel}"/> -->
+      <dynamics damping="${joint_damping}"/>
+    </joint>
+   <link name="${name}_link_6_l">
       <inertial>
         <origin xyz="0 0 0" rpy="0 0 0"/>
@@ -443,5 +497,5 @@
       </collision>
     </link>
-    <!-- joint between link_6_l and link_7_l -->
+   <!-- joint between link_6_l and link_7_l -->
     <joint name="${name}_joint_6_l" type="revolute">
       <parent link="${name}_link_6_l"/>
@@ -451,7 +505,11 @@
       <limit lower="${-229 * PI / 180}" upper="${229 * PI / 180}"
              effort="${max_effort}" velocity="${400 * PI / 180}" />
-      <dynamics damping="${joint_damping}"/>
-    </joint>
-    <link name="${name}_link_7_l">
+      <!--   <safety_controller soft_lower_limit="${-168 * M_PI / 180}"
+           soft_upper_limit="${168 * M_PI / 180}"
+           k_position="${safety_controller_k_pos}"
+           k_velocity="${safety_controller_k_vel}"/> -->
+      <dynamics damping="${joint_damping}"/>
+    </joint>
+   <link name="${name}_link_7_l">
       <inertial>
         <origin xyz="0 0 0" rpy="0 0 0"/>

Commit message: Modifying the URDF a bit to interface YuMi with the pedestals

File: yumi_description/urdf/yumi.urdf.xacro (robot description, xacro)
@@ -13,6 +13,15 @@
   <!-- Fix to world just for testing -->
   <link name="world"/>
+  <!-- <xacro:property name="yumi_setup" value="$(arg yumi_base)" /> -->
+  <!-- <xacro:if value="${yumi_setup == 'default'}"> -->
+<!--     <joint name="world_joint" type="fixed">
+      <origin xyz="0 0 0" rpy="0 0 0" />
+      <parent link="world"/>
+      <child link="yumi_body"/>
+    </joint>
+    <xacro:property name="yumi_base" value="world" /> -->
+  <!-- </xacro:if> -->
   <!--yumi-->
-  <xacro:yumi name="yumi" hardware_interface="hardware_interface/$(arg arms_interface)" parent="world">
+  <xacro:yumi name="yumi" hardware_interface="hardware_interface/$(arg arms_interface)" parent="world" >
     <origin xyz="0 0 0.1" rpy="0 0 0" />
   </xacro:yumi>
@@ -25,3 +34,29 @@
     <origin xyz="0 0 0.007" rpy="0 0 ${PI}" />
   </xacro:yumi_servo_gripper>
+<!--   <xacro:if value="${yumi_base == 'automed_pedestal'}">
+    <xacro:property name="pedestal_height" value="0.28" />
+    <xacro:property name="pedestal_offset_x" value="0.32" />
+    <xacro:property name="yumi_offset_x" value="0.06" />
+    <xacro:property name="yumi_height" value="0.25" />
+    <joint name="ridgeback_base_to_pedestal" type="fixed">
+      <origin rpy="0 0 ${PI}" xyz="${pedestal_offset_x} 0 ${pedestal_height}" />
+      <parent link="base_link" />
+      <child link="yumi_pedestal" />
+    </joint>
+    <link name="yumi_pedestal">
+      <visual>
+        <origin xyz="0 0 0" rpy="0 0 ${PI}" />
+        <geometry>
+          <mesh filename="package://yumi_description/meshes/accesories/KTH_AutoMed_Aluflex_pedestal.stl"/>
+        </geometry>
+        <material name="Light_Gray" />
+      </visual>
+    </link>
+    <joint name="pedestal_to_yumi" type="fixed">
+      <origin rpy="0 0 ${PI}" xyz="${yumi_offset_x} 0 ${yumi_height}" />
+      <parent link="yumi_pedestal" />
+      <child link="yumi_body" />
+    </joint>
+  </xacro:if>
+ -->
 </robot>
