Commit message: Improved the URDF syntax a bit, and added configurations for the FACT and AUTOMED projects, including the metal table, kinect, etc

File: yumi_description/urdf/yumi.urdf.xacro (robot description, xacro)
@@ -11,17 +11,6 @@
   <!-- Import Gazebo plugins -->
   <xacro:include filename="$(find yumi_description)/urdf/Gazebo/gazebo.urdf.xacro"/>
-  <!-- Fix to world just for testing -->
-  <link name="world"/>
-  <!-- <xacro:property name="yumi_setup" value="$(arg yumi_base)" /> -->
-  <!-- <xacro:if value="${yumi_setup == 'default'}"> -->
-<!--     <joint name="world_joint" type="fixed">
-      <origin xyz="0 0 0" rpy="0 0 0" />
-      <parent link="world"/>
-      <child link="yumi_body"/>
-    </joint>
-    <xacro:property name="yumi_base" value="world" /> -->
-  <!-- </xacro:if> -->
   <!--yumi-->
-  <xacro:yumi name="yumi" hardware_interface="hardware_interface/$(arg arms_interface)" parent="world" >
+  <xacro:yumi name="yumi" hardware_interface="hardware_interface/$(arg arms_interface)" parent="${yumi_parent}" >
     <origin xyz="0 0 0.1" rpy="0 0 0" />
   </xacro:yumi>
@@ -34,29 +23,147 @@
     <origin xyz="0 0 0.007" rpy="0 0 ${PI}" />
   </xacro:yumi_servo_gripper>
-<!--   <xacro:if value="${yumi_base == 'automed_pedestal'}">
-    <xacro:property name="pedestal_height" value="0.28" />
-    <xacro:property name="pedestal_offset_x" value="0.32" />
-    <xacro:property name="yumi_offset_x" value="0.06" />
-    <xacro:property name="yumi_height" value="0.25" />
-    <joint name="ridgeback_base_to_pedestal" type="fixed">
-      <origin rpy="0 0 ${PI}" xyz="${pedestal_offset_x} 0 ${pedestal_height}" />
-      <parent link="base_link" />
+  <xacro:property name="yumi_setup" value="$(arg yumi_base)" />
+  <xacro:if value="${yumi_setup == 'default'}">
+    <xacro:property name="yumi_parent" value="world" />
+    <link name="world"/>
+    <joint name="world_joint" type="fixed">
+      <origin xyz="0 0 0.1" rpy="0 0 0" />
+      <parent link="world"/>
+      <child link="yumi_body"/>
+    </joint>
+  </xacro:if>
+  <xacro:if value="${yumi_setup == 'automed'}">
+    <xacro:property name="pedestal_height" value="0.92" />
+    <xacro:property name="pedestal_xrotation_fix" value="${- PI / 2.0}" />
+    <xacro:property name="pedestal_zrotation_fix" value="${PI}" />
+    <xacro:property name="yumi_offset_x" value="-0.0625" />
+    <xacro:property name="yumi_height" value="0.04" />
+    <xacro:property name="yumi_parent" value="yumi_pedestal" />
+    <link name="world"/>
+    <joint name="world_to_pedestal" type="fixed">
+      <origin rpy="0 0 0" xyz="0 0 ${pedestal_height}" />
+      <parent link="world" />
+      <child link="yumi_pedestal" />
+    </joint>
+    <link name="yumi_pedestal">
+<!--       <collision>
+        <origin xyz="0 0 0" rpy="${pedestal_xrotation_fix} 0 ${pedestal_zrotation_fix}" />
+        <geometry>
+          <mesh scale="0.001 0.001 0.001" filename="package://yumi_description/meshes/accesories/KTH_AutoMed_Aluflex_pedestal.stl"/>
+        </geometry>
+        <material name="Grey" />
+      </collision> -->
+      <visual>
+        <origin xyz="0 0 0" rpy="${pedestal_xrotation_fix} 0 ${pedestal_zrotation_fix}" />
+        <geometry>
+          <mesh scale="0.001 0.001 0.001" filename="package://yumi_description/meshes/accesories/KTH_AutoMed_Aluflex_pedestal.stl"/>
+        </geometry>
+        <material name="Grey" />
+      </visual>
+    </link>
+    <joint name="pedestal_to_yumi" type="fixed">
+      <origin rpy="0 0 0" xyz="${yumi_offset_x} 0 ${yumi_height}" />
+      <parent link="yumi_pedestal" />
+      <child link="yumi_body" />
+    </joint>
+  </xacro:if>
+  <xacro:if value="${yumi_setup == 'fact'}">
+    <xacro:property name="pedestal_height" value="0.92" />
+    <xacro:property name="pedestal_xrotation_fix" value="${- PI / 2.0}" />
+    <xacro:property name="pedestal_zrotation_fix" value="${PI}" />
+    <xacro:property name="yumi_offset_x" value="-0.0625" />
+    <xacro:property name="yumi_height" value="0.04" />
+    <xacro:property name="yumi_parent" value="yumi_pedestal" />
+    <xacro:property name="kinect_zrotation_fix" value="${- PI / 2.0}" />
+    <link name="world"/>
+    <joint name="world_to_pedestal" type="fixed">
+      <origin rpy="0 0 0" xyz="0 0 ${pedestal_height}" />
+      <parent link="world" />
       <child link="yumi_pedestal" />
     </joint>
     <link name="yumi_pedestal">
       <visual>
-        <origin xyz="0 0 0" rpy="0 0 ${PI}" />
+        <origin xyz="0 0 0" rpy="${pedestal_xrotation_fix} 0 ${pedestal_zrotation_fix}" />
         <geometry>
-          <mesh filename="package://yumi_description/meshes/accesories/KTH_AutoMed_Aluflex_pedestal.stl"/>
+          <mesh scale="0.001 0.001 0.001" filename="package://yumi_description/meshes/accesories/KTH_AutoMed_Aluflex_pedestal.stl"/>
         </geometry>
-        <material name="Light_Gray" />
+        <material name="Grey" />
       </visual>
     </link>
+    <joint name="pedestal_to_table" type="fixed">
+      <origin rpy="0 0 0" xyz="0.235 0 ${yumi_height}" />
+      <parent link="yumi_pedestal" />
+      <child link="table" />
+    </joint>
+    <link name="table">
+        <visual>
+          <origin xyz="0 0 0" rpy="0 0 0" />
+          <geometry>
+            <box size="0.6 0.6 0.02" />
+          </geometry>
+          <material name="Grey" />
+        </visual>
+    </link>
     <joint name="pedestal_to_yumi" type="fixed">
-      <origin rpy="0 0 ${PI}" xyz="${yumi_offset_x} 0 ${yumi_height}" />
+      <origin rpy="0 0 0" xyz="${yumi_offset_x} 0 ${yumi_height+0.02}" />
       <parent link="yumi_pedestal" />
       <child link="yumi_body" />
     </joint>
+    <link name="kinect2">
+      <visual>
+        <origin xyz="0 0 0" rpy="0 0 0" />
+        <geometry>
+          <mesh scale="0.001 0.001 0.001" filename="package://yumi_description/meshes/accesories/KinectXboxOne.stl"/>
+        </geometry>
+        <material name="Black" />
+      </visual>
+    </link>
+    <link name="left_kinect_base">
+        <visual>
+          <origin xyz="0 0 0" rpy="0 0 0" />
+          <geometry>
+            <box size="0.4 0.02 0.02" />
+          </geometry>
+          <material name="Grey" />
+        </visual>
+    </link>
+    <link name="right_kinect_base">
+        <visual>
+          <origin xyz="0 0 0" rpy="0 0 0" />
+          <geometry>
+            <box size="0.4 0.02 0.02" />
+          </geometry>
+          <material name="Grey" />
+        </visual>
+    </link>
+    <link name="middle_kinect_base">
+        <visual>
+          <origin xyz="0 0 0" rpy="0 0 0" />
+          <geometry>
+            <box size="0.4 0.02 0.02" />
+          </geometry>
+          <material name="Grey" />
+        </visual>
+    </link>
+     <joint name="kinect2_to_right_kinect_base" type="fixed">
+      <origin rpy="0 ${-PI/6} 0.17" xyz="0.1 -0.03 0.56" />
+      <parent link="yumi_body" />
+      <child link="right_kinect_base" />
+    </joint>
+    <joint name="kinect2_to_left_kinect_base" type="fixed">
+      <origin rpy="0 ${-PI/6} -0.17" xyz="0.1 0.03 0.56" />
+      <parent link="yumi_body" />
+      <child link="left_kinect_base" />
+    </joint>
+    <joint name="yumi_to_middle_kinect_base" type="fixed">
+      <origin rpy="0 ${-PI/6} 0" xyz="0.05 0 0.56" />
+      <parent link="yumi_body" />
+      <child link="middle_kinect_base" />
+    </joint>
+    <joint name="middle_kinect_base_to_kinect2" type="fixed">
+      <origin rpy="${-PI/2} 0 ${kinect_zrotation_fix}" xyz="0.2 0 0" />
+      <parent link="middle_kinect_base" />
+      <child link="kinect2" />
+    </joint>
   </xacro:if>
- -->
 </robot>

File: yumi_description/urdf/yumi.xacro (robot description, xacro)
@@ -9,12 +9,4 @@
   <xacro:property name="max_effort" value="300"/>
   <xacro:macro name="yumi" params="parent name hardware_interface *origin">
-    <xacro:if value="${parent == 'world'}">
-      <!--joint between world and body-->
-      <joint name="world_joint" type="fixed">
-        <xacro:insert_block name="origin"/>
-        <parent link="world"/>
-        <child link="${name}_body"/>
-      </joint>
-    </xacro:if>
     <link name="${name}_body">
       <inertial>

Commit message: Updating launch files to comply with URDF changes from yesterday

File: yumi_description/urdf/yumi.urdf.xacro (robot description, xacro)
@@ -23,5 +23,5 @@
     <origin xyz="0 0 0.007" rpy="0 0 ${PI}" />
   </xacro:yumi_servo_gripper>
-  <xacro:property name="yumi_setup" value="$(arg yumi_base)" />
+  <xacro:property name="yumi_setup" value="$(arg yumi_setup)" />
   <xacro:if value="${yumi_setup == 'default'}">
     <xacro:property name="yumi_parent" value="world" />
@@ -33,5 +33,5 @@
     </joint>
   </xacro:if>
-  <xacro:if value="${yumi_setup == 'automed'}">
+  <xacro:if value="${yumi_setup == 'AUTOMED'}">
     <xacro:property name="pedestal_height" value="0.92" />
     <xacro:property name="pedestal_xrotation_fix" value="${- PI / 2.0}" />
@@ -68,5 +68,5 @@
     </joint>
   </xacro:if>
-  <xacro:if value="${yumi_setup == 'fact'}">
+  <xacro:if value="${yumi_setup == 'FACT'}">
     <xacro:property name="pedestal_height" value="0.92" />
     <xacro:property name="pedestal_xrotation_fix" value="${- PI / 2.0}" />

Commit message: reverting to old school yumi setup. alternative setups are now in a new xacro

File: yumi_description/urdf/yumi.urdf.xacro (robot description, xacro)
@@ -23,6 +23,4 @@
     <origin xyz="0 0 0.007" rpy="0 0 ${PI}" />
   </xacro:yumi_servo_gripper>
-  <xacro:property name="yumi_setup" value="$(arg yumi_setup)" />
-  <xacro:if value="${yumi_setup == 'default'}">
     <xacro:property name="yumi_parent" value="world" />
     <link name="world"/>
@@ -32,138 +30,3 @@
       <origin xyz="0 0 0.1" rpy="0 0 0" />
     </joint>
-  </xacro:if>
-  <xacro:if value="${yumi_setup == 'AUTOMED'}">
-    <xacro:property name="pedestal_height" value="0.92" />
-    <xacro:property name="pedestal_xrotation_fix" value="${- PI / 2.0}" />
-    <xacro:property name="pedestal_zrotation_fix" value="${PI}" />
-    <xacro:property name="yumi_offset_x" value="-0.0625" />
-    <xacro:property name="yumi_height" value="0.04" />
-    <xacro:property name="yumi_parent" value="yumi_pedestal" />
-    <link name="world"/>
-    <joint name="world_to_pedestal" type="fixed">
-      <parent link="world" />
-      <child link="yumi_pedestal" />
-      <origin rpy="0 0 0" xyz="0 0 ${pedestal_height}" />
-    </joint>
-    <link name="yumi_pedestal">
-<!--       <collision>
-        <origin xyz="0 0 0" rpy="${pedestal_xrotation_fix} 0 ${pedestal_zrotation_fix}" />
-        <geometry>
-          <mesh scale="0.001 0.001 0.001" filename="package://yumi_description/meshes/accesories/KTH_AutoMed_Aluflex_pedestal.stl"/>
-        </geometry>
-        <material name="Grey" />
-      </collision> -->
-      <visual>
-        <origin xyz="0 0 0" rpy="${pedestal_xrotation_fix} 0 ${pedestal_zrotation_fix}" />
-        <geometry>
-          <mesh scale="0.001 0.001 0.001" filename="package://yumi_description/meshes/accesories/KTH_AutoMed_Aluflex_pedestal.stl"/>
-        </geometry>
-        <material name="Grey" />
-      </visual>
-    </link>
-    <joint name="pedestal_to_yumi" type="fixed">
-      <parent link="yumi_pedestal" />
-      <child link="yumi_base_link" />
-      <origin rpy="0 0 0" xyz="${yumi_offset_x} 0 ${yumi_height}" />
-    </joint>
-  </xacro:if>
-  <xacro:if value="${yumi_setup == 'FACT'}">
-    <xacro:property name="pedestal_height" value="0.92" />
-    <xacro:property name="pedestal_xrotation_fix" value="${- PI / 2.0}" />
-    <xacro:property name="pedestal_zrotation_fix" value="${PI}" />
-    <xacro:property name="yumi_offset_x" value="-0.0625" />
-    <xacro:property name="yumi_height" value="0.04" />
-    <xacro:property name="yumi_parent" value="yumi_pedestal" />
-    <xacro:property name="kinect_zrotation_fix" value="${- PI / 2.0}" />
-    <link name="world"/>
-    <joint name="world_to_pedestal" type="fixed">
-      <parent link="world" />
-      <child link="yumi_pedestal" />
-      <origin rpy="0 0 0" xyz="0 0 ${pedestal_height}" />
-    </joint>
-    <link name="yumi_pedestal">
-      <visual>
-        <origin xyz="0 0 0" rpy="${pedestal_xrotation_fix} 0 ${pedestal_zrotation_fix}" />
-        <geometry>
-          <mesh scale="0.001 0.001 0.001" filename="package://yumi_description/meshes/accesories/KTH_AutoMed_Aluflex_pedestal.stl"/>
-        </geometry>
-        <material name="Grey" />
-      </visual>
-    </link>
-    <joint name="pedestal_to_table" type="fixed">
-      <parent link="yumi_pedestal" />
-      <child link="table" />
-      <origin rpy="0 0 0" xyz="0.235 0 ${yumi_height}" />
-    </joint>
-    <link name="table">
-        <visual>
-          <origin xyz="0 0 0" rpy="0 0 0" />
-          <geometry>
-            <box size="0.6 0.6 0.02" />
-          </geometry>
-          <material name="Grey" />
-        </visual>
-    </link>
-    <joint name="pedestal_to_yumi" type="fixed">
-      <parent link="yumi_pedestal" />
-      <child link="yumi_base_link" />
-      <origin rpy="0 0 0" xyz="${yumi_offset_x} 0 ${yumi_height+0.02}" />
-    </joint>
-    <link name="kinect2">
-      <visual>
-        <origin xyz="0 0 0" rpy="0 0 0" />
-        <geometry>
-          <mesh scale="0.001 0.001 0.001" filename="package://yumi_description/meshes/accesories/KinectXboxOne.stl"/>
-        </geometry>
-        <material name="Black" />
-      </visual>
-    </link>
-    <link name="left_kinect_base">
-        <visual>
-          <origin xyz="0 0 0" rpy="0 0 0" />
-          <geometry>
-            <box size="0.4 0.02 0.02" />
-          </geometry>
-          <material name="Grey" />
-        </visual>
-    </link>
-    <link name="right_kinect_base">
-        <visual>
-          <origin xyz="0 0 0" rpy="0 0 0" />
-          <geometry>
-            <box size="0.4 0.02 0.02" />
-          </geometry>
-          <material name="Grey" />
-        </visual>
-    </link>
-    <link name="middle_kinect_base">
-        <visual>
-          <origin xyz="0 0 0" rpy="0 0 0" />
-          <geometry>
-            <box size="0.4 0.02 0.02" />
-          </geometry>
-          <material name="Grey" />
-        </visual>
-    </link>
-     <joint name="kinect2_to_right_kinect_base" type="fixed">
-      <parent link="yumi_base_link" />
-      <child link="right_kinect_base" />
-      <origin rpy="0 ${-PI/6} 0.17" xyz="0.1 -0.03 0.56" />
-    </joint>
-    <joint name="kinect2_to_left_kinect_base" type="fixed">
-      <parent link="yumi_base_link" />
-      <child link="left_kinect_base" />
-      <origin rpy="0 ${-PI/6} -0.17" xyz="0.1 0.03 0.56" />
-    </joint>
-    <joint name="yumi_to_middle_kinect_base" type="fixed">
-      <parent link="yumi_base_link" />
-      <child link="middle_kinect_base" />
-      <origin rpy="0 ${-PI/6} 0" xyz="0.05 0 0.56" />
-    </joint>
-    <joint name="middle_kinect_base_to_kinect2" type="fixed">
-      <parent link="middle_kinect_base" />
-      <child link="kinect2" />
-      <origin rpy="${-PI/2} 0 ${kinect_zrotation_fix}" xyz="0.2 0 0" />
-    </joint>
-  </xacro:if>
 </robot>

Commit message: Added extra features

File: yumi_description/urdf/yumi.urdf.xacro (robot description, xacro)
@@ -15,5 +15,5 @@
   <!-- Fix to world just for testing -->
   <link name="world"/>
-  <xacro:yumi_table parent="world" table_height="0.6"/>
+  <xacro:yumi_table parent="world" table_height="0.1"/>
   <!--yumi-->
   <xacro:yumi name="yumi" hardware_interface="$(arg prefix)" parent="world">

File: yumi_description/urdf/yumi_table.urdf.xacro (robot description, xacro)
@@ -3,7 +3,7 @@
   <!-- <property name="table_height" value="0.55" /> -->
   <property name="table_width" value="1.08" />
-  <property name="table_depth" value="1.08" />
+  <property name="table_depth" value="1.3" />
   <property name="leg_radius" value="0.02" />
-  <property name="table_x" value="0.0" />
+  <property name="table_x" value="0.3" />
   <property name="table_y" value="0.0" />
   <property name="table_z" value="0.0" />
@@ -45,5 +45,5 @@
       <kd>1.0</kd>
     </gazebo>
-    <joint name="leg1_joint" type="fixed" >
+<!--     <joint name="leg1_joint" type="fixed" >
       <parent link="table_top_link" />
       <origin xyz="${table_x+table_width/2} ${table_y+table_depth/2} ${table_z+table_height}" rpy="0 0 0" />
@@ -185,4 +185,5 @@
       <canonicalBody>table_top_link</canonicalBody>
     </gazebo>
-  </xacro:macro>
+ -->
+</xacro:macro>
 </robot>

Commit message: Added the box

File: yumi_description/urdf/yumi.urdf.xacro (robot description, xacro)
@@ -15,5 +15,5 @@
   <!-- Fix to world just for testing -->
   <link name="world"/>
-  <xacro:yumi_table parent="world" table_height="0.1"/>
+  <xacro:yumi_table parent="world" table_height="0.125"/>
   <!--yumi-->
   <xacro:yumi name="yumi" hardware_interface="$(arg prefix)" parent="world">

File: yumi_description/urdf/yumi_table.urdf.xacro (robot description, xacro)
@@ -8,6 +8,21 @@
   <property name="table_y" value="0.0" />
   <property name="table_z" value="0.0" />
+  <property name="box_x" value="0.3" />
+  <property name="box_y" value="-0.05" />
+  <property name="box_z" value="0" />
+  <property name="box_depth" value="0.075" />
+  <property name="box_height" value="0.12" />
+  <property name="box_width" value="0.021" />
   <property name="table_top_thickness" value="0.02"/>
   <property name="M_PI" value="3.1415926535897931" />
+  <material name="blue">
+    <color rgba="0 0 1 1"/>
+  </material>
+  <material name="black">
+    <color rgba="0 0 0 1"/>
+  </material>
+  <material name="white">
+    <color rgba="1 1 1 1"/>
+  </material>
   <!-- tabletop height is .55+.01+.025=.585 -->
   <xacro:macro name="yumi_table" params="parent table_height">
@@ -30,4 +45,5 @@
           <box size="${table_width} ${table_depth} ${table_top_thickness}" />
         </geometry>
+        <material name="black"/>
       </visual>
       <collision>
@@ -50,4 +66,33 @@
       <self_collide>1</self_collide>
     </gazebo>
+    <joint name="table_box_joint" type="fixed">
+      <origin xyz="0 0 0" />
+      <parent link="${parent}"/>
+      <child link="boxx"/>
+    </joint>
+    <link name="boxx">
+      <inertial>
+        <mass value="1.0" />
+        <origin xyz="${box_x} ${box_y} ${box_z+table_z+table_height+table_top_thickness+box_height/2}" />
+        <inertia ixx="1" ixy="0"  ixz="0"
+         iyy="1" iyz="0"
+         izz="1" />
+       </inertial>
+       <visual>
+        <origin xyz="${box_x} ${box_y} ${table_height+table_top_thickness+box_height/2-0.02}" />
+        <geometry>
+          <box size="${box_depth} ${box_width} ${box_height}" />
+        </geometry>
+        <material name="white"/>
+      </visual>
+    </link>
+    <gazebo reference="boxx">
+      <material>Gazebo/Grey</material>
+      <mu1>50.0</mu1>
+      <mu2>50.0</mu2>
+      <kp>1000000.0</kp>
+      <kd>1.0</kd>
+      <self_collide>1</self_collide>
+    </gazebo>
 <!--     <joint name="leg1_joint" type="fixed" >
       <parent link="table_top_link" />
