Commit message: Fixed collisions

File: yumi_description/urdf/yumi_table.urdf.xacro (robot description, xacro)
@@ -5,8 +5,8 @@
   <property name="table_depth" value="1.3" />
   <property name="leg_radius" value="0.02" />
-  <property name="table_x" value="0.3" />
+  <property name="table_x" value="0.68" />
   <property name="table_y" value="0.0" />
   <property name="table_z" value="0.0" />
-  <property name="table_top_thickness" value="0.05"/>
+  <property name="table_top_thickness" value="0.02"/>
   <property name="M_PI" value="3.1415926535897931" />
   <!-- tabletop height is .55+.01+.025=.585 -->
@@ -37,11 +37,16 @@
         </geometry>
       </collision>
+      <inertial>
+        <mass value="10"/>
+        <inertial ixx="1.0" ixy="0.0" ixz="0.0" iyy="1.0" iyz="0.0" izz="1.0"/>
+      </inertial>
     </link>
     <gazebo reference="table_top_link">
-      <material>Gazebo/Wood</material>
+      <material>Gazebo/Grey</material>
       <mu1>50.0</mu1>
       <mu2>50.0</mu2>
       <kp>1000000.0</kp>
       <kd>1.0</kd>
+      <self_collide>1</self_collide>
     </gazebo>
 <!--     <joint name="leg1_joint" type="fixed" >

Commit message: Work in progress

File: yumi_description/urdf/yumi_table.urdf.xacro (robot description, xacro)
@@ -2,11 +2,11 @@
 <robot name="table" xmlns:xacro="http://www.ros.org/wiki/xacro">
   <!-- <property name="table_height" value="0.55" /> -->
-  <property name="table_width" value="1.08" />
-  <property name="table_depth" value="1.3" />
+  <property name="table_width" value="1.2" />
+  <property name="table_depth" value="1.4" />
   <property name="leg_radius" value="0.02" />
   <property name="table_x" value="0.3" />
   <property name="table_y" value="0.0" />
   <property name="table_z" value="0.0" />
-  <property name="table_top_thickness" value="0.05"/>
+  <property name="table_top_thickness" value="0.1"/>
   <property name="M_PI" value="3.1415926535897931" />
   <!-- tabletop height is .55+.01+.025=.585 -->
@@ -39,5 +39,5 @@
     </link>
     <gazebo reference="table_top_link">
-      <material>Gazebo/Wood</material>
+      <material>Gazebo/Grey</material>
       <mu1>50.0</mu1>
       <mu2>50.0</mu2>

Commit message: Work in progress

File: yumi_description/urdf/yumi_table.urdf.xacro (robot description, xacro)
@@ -5,9 +5,15 @@
   <property name="table_depth" value="1.4" />
   <property name="leg_radius" value="0.02" />
-  <property name="table_x" value="0.68" />
+  <property name="table_x" value="0.74" />
   <property name="table_y" value="0.0" />
   <property name="table_z" value="0.0" />
   <property name="table_top_thickness" value="0.02"/>
   <property name="M_PI" value="3.1415926535897931" />
+  <material name="blue">
+    <color rgba="0 0 1 1"/>
+  </material>
+  <material name="black">
+    <color rgba="0 0 0 1"/>
+  </material>
   <!-- tabletop height is .55+.01+.025=.585 -->
   <xacro:macro name="yumi_table" params="parent table_height">
@@ -30,4 +36,5 @@
           <box size="${table_width} ${table_depth} ${table_top_thickness}" />
         </geometry>
+        <material name="black"/>
       </visual>
       <collision>
@@ -190,5 +197,5 @@
       <canonicalBody>table_top_link</canonicalBody>
     </gazebo>
- -->
+  -->
 </xacro:macro>
 </robot>
