Commit message: Added files for the learning branch

File: yumi_description/gazebo/gazebo.urdf.xacro (robot description, xacro)
@@ -6,3 +6,45 @@
     </plugin>
   </gazebo>
+  <gazebo reference="yumi_top_camera_base">
+    <material>Gazebo/red</material>
+  </gazebo>
+  <!-- camera -->
+  <gazebo reference="yumi_top_camera_base">
+   <sensor type="depth" name="camera">
+    <always_on>true</always_on>
+    <update_rate>30.0</update_rate>
+    <camera>
+      <horizontal_fov>1.0471975511965976</horizontal_fov>
+      <image>
+        <format>R8G8B8</format>
+        <width>640</width>
+        <height>480</height>
+      </image>
+      <clip>
+        <near>0.05</near>
+        <far>8.0</far>
+      </clip>
+    </camera>
+    <plugin name="kinect1_camera_controller" filename="libgazebo_ros_openni_kinect.so">
+      <cameraName>kinect1</cameraName>
+      <alwaysOn>true</alwaysOn>
+      <updateRate>30.0</updateRate>
+      <imageTopicName>rgb/image_raw</imageTopicName>
+      <depthImageTopicName>depth/image_raw</depthImageTopicName>
+      <pointCloudTopicName>depth/points</pointCloudTopicName>
+      <cameraInfoTopicName>rgb/camera_info</cameraInfoTopicName>
+      <depthImageCameraInfoTopicName>depth/camera_info</depthImageCameraInfoTopicName>
+      <frameName>yumi_top_camera_base</frameName>
+      <baseline>0.1</baseline>
+      <distortion_k1>0.0</distortion_k1>
+      <distortion_k2>0.0</distortion_k2>
+      <distortion_k3>0.0</distortion_k3>
+      <distortion_t1>0.0</distortion_t1>
+      <distortion_t2>0.0</distortion_t2>
+      <pointCloudCutoff>0.5</pointCloudCutoff>
+      <pointCloudCutoffMax>5.0</pointCloudCutoffMax>
+    </plugin>
+    <visualize>true</visualize>
+  </sensor>
+</gazebo>
 </robot>

File: yumi_description/urdf/yumi_servo_gripper.gazebo.xacro (robot description, xacro)
@@ -2,18 +2,52 @@
 <robot name="yumi_servo_gripper" xmlns:xacro="http://www.ros.org/wiki/xacro">
   <xacro:macro name="yumi_servo_gripper_gazebo" params="name">
-  <!-- Plugin for the mimic o/c joint - AFAIK, that shouldn't be necessary any more starting with Gazebo 3.0 -->
+    <!-- Plugin for the mimic o/c joint - AFAIK, that shouldn't be necessary any more starting with Gazebo 3.0 -->
     <gazebo>
       <plugin name="mimic_plugin" filename="libgazebo_mimic_plugin.so">
        <joint>${name}_joint</joint>
-        <mimicJoint>${name}_joint_m</mimicJoint>
-        <multiplier>1.0</multiplier>
+       <mimicJoint>${name}_joint_m</mimicJoint>
+       <multiplier>1.0</multiplier>
+     </plugin>
+   </gazebo>
+   <!-- body -->
+   <gazebo reference="${name}_base">
+    <material>Gazebo/Light_Grey</material>
+    <mu1>0.2</mu1>
+    <mu2>0.2</mu2>
+  </gazebo>
+  <gazebo reference= "${name}_finger_r">
+    <sensor name="${name}_finger_r_bumper" type="contact">
+      <always_on>true</always_on>
+      <update_rate>100</update_rate>
+      <contact>
+        <collision>${name}_finger_r_collision</collision>
+        <!-- <topic>/${name}/fr/contact_forces</topic> -->
+      </contact>
+      <plugin filename="libgazebo_ros_bumper.so" name="${name}_finger_r_plugin">
+        <always_on>1</always_on>
+        <update_rate>100</update_rate>
+        <frameName>${name}_finger_r</frameName>
+        <bumperTopicName>${name}/fr/contact</bumperTopicName>
       </plugin>
-    </gazebo>
-    <!-- body -->
-    <gazebo reference="${name}_base">
-      <material>Gazebo/Light_Grey</material>
-      <mu1>0.2</mu1>
-      <mu2>0.2</mu2>
-    </gazebo>
-  </xacro:macro>
+    </sensor>
+    <material>Gazebo/Orange</material>
+  </gazebo>
+  <gazebo reference= "${name}_finger_l" >
+    <sensor name="${name}_finger_l_bumper" type="contact">
+      <always_on>true</always_on>
+      <update_rate>100</update_rate>
+      <contact>
+        <collision>${name}_finger_l_collision</collision>
+        <!-- <topic>/${name}/fl/contact_forces</topic> -->
+      </contact>
+      <plugin filename="libgazebo_ros_bumper.so" name="${name}_finger_l_plugin">
+        <always_on>true</always_on>
+        <update_rate>100</update_rate>
+        <frameName>${name}_finger_l</frameName>
+        <bumperTopicName>${name}/fl/contact</bumperTopicName>
+      </plugin>
+    </sensor>
+    <material>Gazebo/Blue</material>
+  </gazebo>
+</xacro:macro>
 </robot>

File: yumi_description/urdf/yumi_update.urdf.xacro (robot description, xacro)
@@ -11,24 +11,13 @@
   <!--Import the yumi camera macro -->
   <xacro:include filename="$(find yumi_description)/urdf/yumi_camera.xacro"/>
-  <!--Import the table macro -->
-  <xacro:include filename="$(find yumi_description)/urdf/yumi_table.urdf.xacro"/>
-  <!--Import the box macro -->
-  <!-- <xacro:include filename="$(find yumi_description)/urdf/object.urdf.xacro"/> -->
+  <!--Import the yumi box macro -->
+  <!-- <xacro:include filename="$(find yumi_description)/urdf/box.xacro"/> -->
   <!-- Import Gazebo plugins -->
   <xacro:include filename="$(find yumi_description)/gazebo/gazebo.urdf.xacro"/>
   <!-- Fix to world just for testing -->
   <link name="world"/>
-  <!--Define the table height-->
-  <property name="table_height_from_gound" value="0.89" />
-  <!--table-->
-  <xacro:yumi_table parent="world" table_height="${table_height_from_gound}"/>
-  <!--box-->
-<!--   <xacro:yumi_box parent="table_top_link">
-    <origin xyz="0.5 0 ${table_height_from_gound+0.1}" rpy="0 0 0" />
-  </xacro:yumi_box>
- -->
   <!--yumi-->
-  <xacro:yumi name="yumi" hardware_interface="$(arg prefix)" parent="table_top_link">
-    <origin xyz="0 0 ${table_height_from_gound}" rpy="0 0 0" />
+  <xacro:yumi name="yumi" hardware_interface="$(arg prefix)" parent="world">
+    <origin xyz="0 0 0.1" rpy="0 0 0" />
   </xacro:yumi>
   <!--right gripper-->
@@ -40,6 +29,10 @@
     <origin xyz="0 0 0.007" rpy="0 0 ${PI}" />
   </xacro:yumi_servo_gripper>
-  <xacro:yumi_camera name="yumi_top_camera" parent="table_top_link">
-    <origin xyz="0.883 -0.06 ${0.877+table_height_from_gound}" rpy="3.12 0.795 0.005" />
+  <xacro:yumi_camera name="yumi_top_camera" parent="world">
+    <origin xyz="0.883 -0.06 0.877" rpy="3.12 0.795 0.005" />
   </xacro:yumi_camera>
+<!--   <xacro:yumi_box name="box" parent="world">
+    <origin xyz="0.883 -0.06 0.877" rpy="0 0 0" />
+  </xacro:yumi_box>
+ -->
 </robot>
