Commit message: Organizing yumi_description, and deleting old files

File: yumi_description/urdf/Gazebo/yumi.gazebo.xacro (robot description, xacro)
@@ -2,5 +2,5 @@
 <robot name="yumi" xmlns:xacro="http://www.ros.org/wiki/xacro">
   <xacro:macro name="yumi_gazebo" params="name">
-    <!-- body -->
+    <!-- Gazebo reference frame -->
     <gazebo reference="${name}_body">
       <material>Gazebo/Ivory</material>

File: yumi_description/urdf/Grippers/yumi_servo_gripper.xacro (robot description, xacro)
@@ -2,9 +2,7 @@
 <robot name="yumi" xmlns:xacro="http://www.ros.org/wiki/xacro">
     <!-- Import all Gazebo-customization elements, including Gazebo colors -->
-    <xacro:include filename="$(find yumi_description)/urdf/yumi_servo_gripper.gazebo.xacro" />
+    <xacro:include filename="$(find yumi_description)/urdf/Grippers/yumi_servo_gripper.gazebo.xacro" />
     <!-- Import Transmissions -->
-    <xacro:include filename="$(find yumi_description)/urdf/yumi_servo_gripper.transmission.xacro" />
-    <!-- Include Utilities -->
-    <xacro:include filename="$(find yumi_description)/urdf/utilities.xacro" />
+    <xacro:include filename="$(find yumi_description)/urdf/Grippers/yumi_servo_gripper.transmission.xacro" />
     <!-- some constants -->
     <xacro:property name="joint_damping" value="0.5" />

File: yumi_description/urdf/yumi.urdf.xacro (robot description, xacro)
@@ -2,13 +2,13 @@
 <robot name="yumi" xmlns:xacro="http://www.ros.org/wiki/xacro">
   <!-- Import Rviz colors -->
-  <xacro:include filename="$(find yumi_description)/urdf/materials.xacro" />
+  <xacro:include filename="$(find yumi_description)/urdf/Util/materials.xacro" />
   <!-- Import utilities -->
-  <xacro:include filename="$(find yumi_description)/urdf/utilities.xacro" />
+  <xacro:include filename="$(find yumi_description)/urdf/Util/utilities.xacro" />
   <!--Import the yumi macro -->
   <xacro:include filename="$(find yumi_description)/urdf/yumi.xacro"/>
   <!--Import the yumi servo gripper macro -->
-  <xacro:include filename="$(find yumi_description)/urdf/yumi_servo_gripper.xacro"/>
+  <xacro:include filename="$(find yumi_description)/urdf/Grippers/yumi_servo_gripper.xacro"/>
   <!-- Import Gazebo plugins -->
-  <xacro:include filename="$(find yumi_description)/gazebo/gazebo.urdf.xacro"/>
+  <xacro:include filename="$(find yumi_description)/urdf/Gazebo/gazebo.urdf.xacro"/>
   <!-- Fix to world just for testing -->
   <link name="world"/>

File: yumi_description/urdf/yumi.xacro (robot description, xacro)
@@ -2,9 +2,7 @@
 <robot name="yumi" xmlns:xacro="http://www.ros.org/wiki/xacro">
   <!-- Import all Gazebo-customization elements, including Gazebo colors -->
-  <xacro:include filename="$(find yumi_description)/urdf/yumi.gazebo.xacro" />
+  <xacro:include filename="$(find yumi_description)/urdf/Gazebo/yumi.gazebo.xacro" />
   <!-- Import Transmissions -->
   <xacro:include filename="$(find yumi_description)/urdf/yumi.transmission.xacro" />
-  <!-- Include Utilities -->
-  <xacro:include filename="$(find yumi_description)/urdf/utilities.xacro" />
   <!-- some constants -->
  <!-- <xacro:property name="safety_controller_k_pos" value="100" />
@@ -12,5 +10,5 @@
   <xacro:property name="joint_damping" value="0.5" />
   <xacro:property name="max_effort" value="300"/>
-  <xacro:macro name="yumi" params="parent name hardware_interface *origin">
+  <xacro:macro name="yumi" params="name parent hardware_interface *origin">
     <!--joint between {parent} and body-->
     <joint name="${parent}_joint" type="fixed">

File: yumi_description/urdf/yumi_nogrippers.urdf.xacro (robot description, xacro)
@@ -2,11 +2,11 @@
 <robot name="yumi" xmlns:xacro="http://www.ros.org/wiki/xacro">
   <!-- Import Rviz colors -->
-  <xacro:include filename="$(find yumi_description)/urdf/materials.xacro" />
+  <xacro:include filename="$(find yumi_description)/urdf/Util/materials.xacro" />
   <!-- Import utilities -->
-  <xacro:include filename="$(find yumi_description)/urdf/utilities.xacro" />
+  <xacro:include filename="$(find yumi_description)/urdf/Util/utilities.xacro" />
   <!--Import the yumi macro -->
   <xacro:include filename="$(find yumi_description)/urdf/yumi.xacro"/>
- <!-- Import Gazebo plugins -->
-  <xacro:include filename="$(find yumi_description)/gazebo/gazebo.urdf.xacro"/>
+  <!-- Import Gazebo plugins -->
+  <xacro:include filename="$(find yumi_description)/urdf/Gazebo/gazebo.urdf.xacro"/>
   <!-- Fix to world just for testing -->
   <link name="world"/>
